File: files/pcb/kicad/AM2321.sch (KiCad schematic (older format))
At the start: 0 parts

Commit message: 回路図更新
温度湿度センサ
大気圧センサ
輝度センサ
Parts:
- added IC?: AM2321, symbol IC_4PIN
Connections:
- net labels added: +5V, GND, SCL, SDA
- wire segments 0 -> 6
Changed lines of the file:
@@
 $Descr A4 11693 8268
 encoding utf-8
-Sheet 1 12
+Sheet 12 12
 Title ""
 Date "23 aug 2014"
@@
 Comment4 ""
 $EndDescr
+$Comp
+L IC_4PIN IC?
+U 1 1 53F95897
+P 6150 3850
+F 0 "IC?" H 6150 4100 39  0000 C CNN
+F 1 "AM2321" H 6150 3850 39  0000 C CNN
+F 2 "" H 6150 3850 60  0000 C CNN
+F 3 "" H 6150 3850 60  0000 C CNN
+	1    6150 3850
+	1    0    0    -1
+$EndComp
+$Comp
+L GND #PWR?
+U 1 1 53F958B5
+P 5600 4350
+F 0 "#PWR?" H 5600 4350 30  0001 C CNN
+F 1 "GND" H 5600 4280 30  0001 C CNN
+F 2 "" H 5600 4350 60  0000 C CNN
+F 3 "" H 5600 4350 60  0000 C CNN
+	1    5600 4350
+	1    0    0    -1
+$EndComp
+$Comp
+L +5V #PWR?
+U 1 1 53F958C4
+P 5600 3450
+F 0 "#PWR?" H 5600 3540 20  0001 C CNN
+F 1 "+5V" H 5600 3540 30  0000 C CNN
+F 2 "" H 5600 3450 60  0000 C CNN
+F 3 "" H 5600 3450 60  0000 C CNN
+	1    5600 3450
+	1    0    0    -1
+$EndComp
+Wire Wire Line
+	5700 3700 5600 3700
+Wire Wire Line
+	5600 3700 5600 3450
+Wire Wire Line
+	5700 3900 5600 3900
+Wire Wire Line
+	5600 3900 5600 4350
+Wire Wire Line
+	5000 4000 5700 4000
+Wire Wire Line
+	5700 3800 5000 3800
+Text HLabel 5000 3800 0    60   Input ~ 0
+SDA
+Text HLabel 5000 4000 0    60   Input ~ 0
+SCL
 $EndSCHEMATC

Commit message: 回路図更新、DS1307対応
バスの接続が未
Parts:
- removed IC?: AM2321, symbol IC_4PIN
- added IC12: AM2321, ~, symbol IC_4PIN_S
Changed lines of the file:
@@
 $Descr A4 11693 8268
 encoding utf-8
-Sheet 12 12
+Sheet 13 13
 Title ""
-Date "23 aug 2014"
+Date "24 aug 2014"
 Rev ""
 Comp ""
@@
 $EndDescr
 $Comp
-L IC_4PIN IC?
-U 1 1 53F95897
-P 6150 3850
-F 0 "IC?" H 6150 4100 39  0000 C CNN
-F 1 "AM2321" H 6150 3850 39  0000 C CNN
-F 2 "" H 6150 3850 60  0000 C CNN
-F 3 "" H 6150 3850 60  0000 C CNN
-	1    6150 3850
-	1    0    0    -1
-$EndComp
-$Comp
-L GND #PWR?
+L GND #PWR58
 U 1 1 53F958B5
 P 5600 4350
-F 0 "#PWR?" H 5600 4350 30  0001 C CNN
+F 0 "#PWR58" H 5600 4350 30  0001 C CNN
 F 1 "GND" H 5600 4280 30  0001 C CNN
 F 2 "" H 5600 4350 60  0000 C CNN
@@
 $EndComp
 $Comp
-L +5V #PWR?
+L +5V #PWR57
 U 1 1 53F958C4
 P 5600 3450
-F 0 "#PWR?" H 5600 3540 20  0001 C CNN
+F 0 "#PWR57" H 5600 3540 20  0001 C CNN
 F 1 "+5V" H 5600 3540 30  0000 C CNN
 F 2 "" H 5600 3450 60  0000 C CNN
@@
 Text HLabel 5000 4000 0    60   Input ~ 0
 SCL
+$Comp
+L IC_4PIN_S IC12
+U 1 1 53FABC17
+P 6150 3850
+F 0 "IC12" H 6150 4100 39  0000 C CNN
+F 1 "AM2321" H 6150 3850 39  0000 C CNN
+F 2 "~" H 6100 3800 60  0000 C CNN
+F 3 "~" H 6100 3800 60  0000 C CNN
+	1    6150 3850
+	1    0    0    -1
+$EndComp
 $EndSCHEMATC

Commit message: 部品リスト・パッケージライブラリを更新
Parts:
- renumbered IC12 to IC13
Changed lines of the file:
@@
 $EndDescr
 $Comp
-L GND #PWR068
+L GND #PWR071
 U 1 1 53F958B5
 P 5600 4350
-F 0 "#PWR068" H 5600 4350 30  0001 C CNN
+F 0 "#PWR071" H 5600 4350 30  0001 C CNN
 F 1 "GND" H 5600 4280 30  0001 C CNN
 F 2 "" H 5600 4350 60  0000 C CNN
@@
 $EndComp
 $Comp
-L +5V #PWR069
+L +5V #PWR072
 U 1 1 53F958C4
 P 5600 3450
-F 0 "#PWR069" H 5600 3540 20  0001 C CNN
+F 0 "#PWR072" H 5600 3540 20  0001 C CNN
 F 1 "+5V" H 5600 3540 30  0000 C CNN
 F 2 "" H 5600 3450 60  0000 C CNN
@@
 SCL
 $Comp
-L IC_4PIN_S IC12
+L IC_4PIN_S IC13
 U 1 1 53FABC17
 P 6150 3850
-F 0 "IC12" H 6150 4100 39  0000 C CNN
+F 0 "IC13" H 6150 4100 39  0000 C CNN
 F 1 "AM2321" H 6150 3850 39  0000 C CNN
 F 2 "~" H 6100 3800 60  0000 C CNN

Commit message: 部品リスト完了、PCBに部品を配置
Parts:
- added C19: 0.1u, ~, symbol C
Connections:
- net +5V: now also C19.1
- net GND: now also C19.2
Changed lines of the file:
@@
 Sheet 13 13
 Title ""
-Date "26 aug 2014"
+Date "28 aug 2014"
 Rev ""
 Comp ""
@@
 $EndDescr
 $Comp
-L GND #PWR071
+L GND #PWR072
 U 1 1 53F958B5
-P 5600 4350
-F 0 "#PWR071" H 5600 4350 30  0001 C CNN
-F 1 "GND" H 5600 4280 30  0001 C CNN
-F 2 "" H 5600 4350 60  0000 C CNN
-F 3 "" H 5600 4350 60  0000 C CNN
-	1    5600 4350
+P 5600 4750
+F 0 "#PWR072" H 5600 4750 30  0001 C CNN
+F 1 "GND" H 5600 4680 30  0001 C CNN
+F 2 "" H 5600 4750 60  0000 C CNN
+F 3 "" H 5600 4750 60  0000 C CNN
+	1    5600 4750
 	1    0    0    -1
 $EndComp
 $Comp
-L +5V #PWR072
+L +5V #PWR073
 U 1 1 53F958C4
-P 5600 3450
-F 0 "#PWR072" H 5600 3540 20  0001 C CNN
-F 1 "+5V" H 5600 3540 30  0000 C CNN
-F 2 "" H 5600 3450 60  0000 C CNN
-F 3 "" H 5600 3450 60  0000 C CNN
-	1    5600 3450
+P 5350 3450
+F 0 "#PWR073" H 5350 3540 20  0001 C CNN
+F 1 "+5V" H 5350 3540 30  0000 C CNN
+F 2 "" H 5350 3450 60  0000 C CNN
+F 3 "" H 5350 3450 60  0000 C CNN
+	1    5350 3450
 	1    0    0    -1
 $EndComp
 Wire Wire Line
-	5700 3700 5600 3700
+	5700 3700 5350 3700
 Wire Wire Line
-	5600 3700 5600 3450
+	5350 3450 5350 4100
 Wire Wire Line
 	5700 3900 5600 3900
 Wire Wire Line
-	5600 3900 5600 4350
+	5600 3900 5600 4750
 Wire Wire Line
 	5000 4000 5700 4000
@@
 	1    0    0    -1
 $EndComp
+$Comp
+L C C19
+U 1 1 53FF65D2
+P 5350 4300
+F 0 "C19" H 5350 4400 40  0000 L CNN
+F 1 "0.1u" H 5356 4215 40  0000 L CNN
+F 2 "~" H 5388 4150 30  0000 C CNN
+F 3 "~" H 5350 4300 60  0000 C CNN
+	1    5350 4300
+	1    0    0    -1
+$EndComp
+Connection ~ 5350 3700
+Wire Wire Line
+	5350 4500 5600 4500
+Connection ~ 5600 4500
 $EndSCHEMATC
