File: files/pcb/kicad/LPS331.sch (KiCad schematic (older format))
At the start: 0 parts

Commit message: 回路図更新
温度湿度センサ
大気圧センサ
輝度センサ
Parts:
- added IC?: IC_8PIN, symbol IC_8PIN
Connections:
- new net +5V: IC?.1, IC?.4, IC?.5
- new net GND: IC?.8
- new net SCL: IC?.2
- new net SDA: IC?.3
- no-connect marks 0 -> 2
Other:
- note added: "4:SDO //SLA low bit\n5:CS // IIC/~SPI\n6:int1\n7:int2"
Changed lines of the file:
@@
 $Descr A4 11693 8268
 encoding utf-8
-Sheet 1 12
+Sheet 11 12
 Title ""
 Date "23 aug 2014"
@@
 Comment4 ""
 $EndDescr
+$Comp
+L IC_8PIN IC?
+U 1 1 53F95D31
+P 5950 3850
+F 0 "IC?" H 5950 4100 39  0000 C CNN
+F 1 "IC_8PIN" H 5950 3850 39  0000 C CNN
+F 2 "" H 5950 3750 60  0000 C CNN
+F 3 "" H 5950 3750 60  0000 C CNN
+	1    5950 3850
+	1    0    0    -1
+$EndComp
+$Comp
+L +5V #PWR?
+U 1 1 53F95D40
+P 5300 3400
+F 0 "#PWR?" H 5300 3490 20  0001 C CNN
+F 1 "+5V" H 5300 3490 30  0000 C CNN
+F 2 "" H 5300 3400 60  0000 C CNN
+F 3 "" H 5300 3400 60  0000 C CNN
+	1    5300 3400
+	1    0    0    -1
+$EndComp
+Wire Wire Line
+	5500 3700 5300 3700
+Wire Wire Line
+	5300 3400 5300 3700
+Wire Wire Line
+	5300 3700 5300 4000
+Wire Wire Line
+	6400 3700 6700 3700
+Wire Wire Line
+	6700 3700 6700 4400
+$Comp
+L GND #PWR?
+U 1 1 53F95D58
+P 6700 4400
+F 0 "#PWR?" H 6700 4400 30  0001 C CNN
+F 1 "GND" H 6700 4330 30  0001 C CNN
+F 2 "" H 6700 4400 60  0000 C CNN
+F 3 "" H 6700 4400 60  0000 C CNN
+	1    6700 4400
+	1    0    0    -1
+$EndComp
+Wire Wire Line
+	4850 3800 5500 3800
+Wire Wire Line
+	5500 3900 4850 3900
+Text HLabel 4850 3800 0    60   Input ~ 0
+SCL
+Text HLabel 4850 3900 0    60   Input ~ 0
+SDA
+Wire Wire Line
+	5300 4000 5500 4000
+Connection ~ 5300 3700
+Text Notes 5700 4200 0    39   ~ 0
+4:SDO //SLA low bit\n5:CS // IIC/~SPI\n6:int1\n7:int2
+NoConn ~ 6400 3900
+NoConn ~ 6400 3800
+Wire Wire Line
+	6400 4000 6550 4000
+Wire Wire Line
+	6550 4000 6550 3400
+$Comp
+L +5V #PWR?
+U 1 1 53F95D95
+P 6550 3400
+F 0 "#PWR?" H 6550 3490 20  0001 C CNN
+F 1 "+5V" H 6550 3490 30  0000 C CNN
+F 2 "" H 6550 3400 60  0000 C CNN
+F 3 "" H 6550 3400 60  0000 C CNN
+	1    6550 3400
+	1    0    0    -1
+$EndComp
 $EndSCHEMATC

Commit message: 回路図更新、DS1307対応
バスの接続が未
Parts:
- gave numbers to parts that had none: 1
Changed lines of the file:
@@
 $Descr A4 11693 8268
 encoding utf-8
-Sheet 11 12
+Sheet 12 13
 Title ""
-Date "23 aug 2014"
+Date "24 aug 2014"
 Rev ""
 Comp ""
@@
 $EndDescr
 $Comp
-L IC_8PIN IC?
+L IC_8PIN IC6
 U 1 1 53F95D31
 P 5950 3850
-F 0 "IC?" H 5950 4100 39  0000 C CNN
+F 0 "IC6" H 5950 4100 39  0000 C CNN
 F 1 "IC_8PIN" H 5950 3850 39  0000 C CNN
 F 2 "" H 5950 3750 60  0000 C CNN
@@
 $EndComp
 $Comp
-L +5V #PWR?
+L +5V #PWR54
 U 1 1 53F95D40
 P 5300 3400
-F 0 "#PWR?" H 5300 3490 20  0001 C CNN
+F 0 "#PWR54" H 5300 3490 20  0001 C CNN
 F 1 "+5V" H 5300 3490 30  0000 C CNN
 F 2 "" H 5300 3400 60  0000 C CNN
@@
 	6700 3700 6700 4400
 $Comp
-L GND #PWR?
+L GND #PWR56
 U 1 1 53F95D58
 P 6700 4400
-F 0 "#PWR?" H 6700 4400 30  0001 C CNN
+F 0 "#PWR56" H 6700 4400 30  0001 C CNN
 F 1 "GND" H 6700 4330 30  0001 C CNN
 F 2 "" H 6700 4400 60  0000 C CNN
@@
 	6550 4000 6550 3400
 $Comp
-L +5V #PWR?
+L +5V #PWR55
 U 1 1 53F95D95
 P 6550 3400
-F 0 "#PWR?" H 6550 3490 20  0001 C CNN
+F 0 "#PWR55" H 6550 3490 20  0001 C CNN
 F 1 "+5V" H 6550 3490 30  0000 C CNN
 F 2 "" H 6550 3400 60  0000 C CNN

Commit message: 回路図ERC途中
Changed lines of the file:
@@
 Sheet 12 13
 Title ""
-Date "24 aug 2014"
+Date "25 aug 2014"
 Rev ""
 Comp ""
@@
 $EndComp
 $Comp
-L +5V #PWR54
+L +5V #PWR057
 U 1 1 53F95D40
 P 5300 3400
-F 0 "#PWR54" H 5300 3490 20  0001 C CNN
+F 0 "#PWR057" H 5300 3490 20  0001 C CNN
 F 1 "+5V" H 5300 3490 30  0000 C CNN
 F 2 "" H 5300 3400 60  0000 C CNN
@@
 	5500 3700 5300 3700
 Wire Wire Line
-	5300 3400 5300 3700
-Wire Wire Line
-	5300 3700 5300 4000
+	5300 3400 5300 4000
 Wire Wire Line
 	6400 3700 6700 3700
@@
 	6700 3700 6700 4400
 $Comp
-L GND #PWR56
+L GND #PWR058
 U 1 1 53F95D58
 P 6700 4400
-F 0 "#PWR56" H 6700 4400 30  0001 C CNN
+F 0 "#PWR058" H 6700 4400 30  0001 C CNN
 F 1 "GND" H 6700 4330 30  0001 C CNN
 F 2 "" H 6700 4400 60  0000 C CNN
@@
 	6550 4000 6550 3400
 $Comp
-L +5V #PWR55
+L +5V #PWR059
 U 1 1 53F95D95
 P 6550 3400
-F 0 "#PWR55" H 6550 3490 20  0001 C CNN
+F 0 "#PWR059" H 6550 3490 20  0001 C CNN
 F 1 "+5V" H 6550 3490 30  0000 C CNN
 F 2 "" H 6550 3400 60  0000 C CNN

Commit message: 部品リスト・パッケージライブラリを更新
Parts:
- renumbered IC6 to IC12
Changed lines of the file:
@@
 $EndDescr
 $Comp
-L IC_8PIN IC6
+L IC_8PIN IC12
 U 1 1 53F95D31
 P 5950 3850
-F 0 "IC6" H 5950 4100 39  0000 C CNN
+F 0 "IC12" H 5950 4100 39  0000 C CNN
 F 1 "IC_8PIN" H 5950 3850 39  0000 C CNN
 F 2 "" H 5950 3750 60  0000 C CNN
@@
 $EndComp
 $Comp
-L +5V #PWR065
+L +5V #PWR068
 U 1 1 53F95D40
 P 5300 3400
-F 0 "#PWR065" H 5300 3490 20  0001 C CNN
+F 0 "#PWR068" H 5300 3490 20  0001 C CNN
 F 1 "+5V" H 5300 3490 30  0000 C CNN
 F 2 "" H 5300 3400 60  0000 C CNN
@@
 	6700 3700 6700 4400
 $Comp
-L GND #PWR066
+L GND #PWR069
 U 1 1 53F95D58
 P 6700 4400
-F 0 "#PWR066" H 6700 4400 30  0001 C CNN
+F 0 "#PWR069" H 6700 4400 30  0001 C CNN
 F 1 "GND" H 6700 4330 30  0001 C CNN
 F 2 "" H 6700 4400 60  0000 C CNN
@@
 	6550 4000 6550 3400
 $Comp
-L +5V #PWR067
+L +5V #PWR070
 U 1 1 53F95D95
 P 6550 3400
-F 0 "#PWR067" H 6550 3490 20  0001 C CNN
+F 0 "#PWR070" H 6550 3490 20  0001 C CNN
 F 1 "+5V" H 6550 3490 30  0000 C CNN
 F 2 "" H 6550 3400 60  0000 C CNN

Commit message: 部品リスト完了、PCBに部品を配置
Parts:
- IC12: value IC_8PIN -> LPS331AP
Changed lines of the file:
@@
 Sheet 12 13
 Title ""
-Date "26 aug 2014"
+Date "28 aug 2014"
 Rev ""
 Comp ""
@@
 P 5950 3850
 F 0 "IC12" H 5950 4100 39  0000 C CNN
-F 1 "IC_8PIN" H 5950 3850 39  0000 C CNN
+F 1 "LPS331AP" H 5950 3850 39  0000 C CNN
 F 2 "" H 5950 3750 60  0000 C CNN
 F 3 "" H 5950 3750 60  0000 C CNN
@@
 $EndComp
 $Comp
-L +5V #PWR068
+L +5V #PWR069
 U 1 1 53F95D40
 P 5300 3400
-F 0 "#PWR068" H 5300 3490 20  0001 C CNN
+F 0 "#PWR069" H 5300 3490 20  0001 C CNN
 F 1 "+5V" H 5300 3490 30  0000 C CNN
 F 2 "" H 5300 3400 60  0000 C CNN
@@
 	6700 3700 6700 4400
 $Comp
-L GND #PWR069
+L GND #PWR070
 U 1 1 53F95D58
 P 6700 4400
-F 0 "#PWR069" H 6700 4400 30  0001 C CNN
+F 0 "#PWR070" H 6700 4400 30  0001 C CNN
 F 1 "GND" H 6700 4330 30  0001 C CNN
 F 2 "" H 6700 4400 60  0000 C CNN
@@
 	6550 4000 6550 3400
 $Comp
-L +5V #PWR070
+L +5V #PWR071
 U 1 1 53F95D95
 P 6550 3400
-F 0 "#PWR070" H 6550 3490 20  0001 C CNN
+F 0 "#PWR071" H 6550 3490 20  0001 C CNN
 F 1 "+5V" H 6550 3490 30  0000 C CNN
 F 2 "" H 6550 3400 60  0000 C CNN
