File: files/pcb/kicad/RTC_DS1307.sch (KiCad schematic (older format))
At the start: 8 parts, among them IC11 DS1307, X2 32.768kHz

Commit message: PCB
Connections:
- net +5V: no longer R27.1
- net CLK_PW_H: now reaches D5.2 (K), IC11.3
- net CLK_PW_H: no longer C14.1
- new net 5V_L: R27.1
- new net CLK_PW_L: C14.1
Other:
- moved on the sheet: C14
Changed lines of the file:
@@
 $Descr A4 11693 8268
 encoding utf-8
-Sheet 11 13
+Sheet 10 13
 Title ""
-Date "30 aug 2014"
+Date "31 aug 2014"
 Rev ""
 Comp ""
@@
 L CP1 C14
 U 1 1 53F95FE8
-P 4650 4500
-F 0 "C14" H 4700 4600 50  0000 L CNN
-F 1 "5.5V 0.1F" H 4700 4400 50  0000 L CNN
-F 2 "~" H 4650 4500 60  0000 C CNN
-F 3 "~" H 4650 4500 60  0000 C CNN
-	1    4650 4500
+P 4750 5450
+F 0 "C14" H 4800 5550 50  0000 L CNN
+F 1 "5.5V 0.1F" H 4800 5350 50  0000 L CNN
+F 2 "~" H 4750 5450 60  0000 C CNN
+F 3 "~" H 4750 5450 60  0000 C CNN
+	1    4750 5450
 	1    0    0    -1
 $EndComp
@@
 $EndComp
 $Comp
-L +5V #PWR062
-U 1 1 53F9602E
-P 4150 3550
-F 0 "#PWR062" H 4150 3640 20  0001 C CNN
-F 1 "+5V" H 4150 3640 30  0000 C CNN
-F 2 "" H 4150 3550 60  0000 C CNN
-F 3 "" H 4150 3550 60  0000 C CNN
-	1    4150 3550
-	1    0    0    -1
-$EndComp
-$Comp
-L GND #PWR063
+L GND #PWR045
 U 1 1 53F96055
 P 4150 4800
-F 0 "#PWR063" H 4150 4800 30  0001 C CNN
+F 0 "#PWR045" H 4150 4800 30  0001 C CNN
 F 1 "GND" H 4150 4730 30  0001 C CNN
 F 2 "" H 4150 4800 60  0000 C CNN
@@
 Wire Wire Line
 	4900 4100 4900 3850
-Wire Wire Line
-	4150 3550 4150 3600
 Wire Wire Line
 	4150 4750 4150 4800
@@
 	6550 4300 7400 4300
 $Comp
-L +5V #PWR064
+L +5V #PWR046
 U 1 1 53F961EF
 P 6700 3400
-F 0 "#PWR064" H 6700 3490 20  0001 C CNN
+F 0 "#PWR046" H 6700 3490 20  0001 C CNN
 F 1 "+5V" H 6700 3490 30  0000 C CNN
 F 2 "" H 6700 3400 60  0000 C CNN
@@
 $EndComp
 $Comp
-L GND #PWR065
+L GND #PWR047
 U 1 1 53F961FF
 P 5500 4450
-F 0 "#PWR065" H 5500 4450 30  0001 C CNN
+F 0 "#PWR047" H 5500 4450 30  0001 C CNN
 F 1 "GND" H 5500 4380 30  0001 C CNN
 F 2 "" H 5500 4450 60  0000 C CNN
@@
 	7150 3400 7150 3500
 $Comp
-L +5V #PWR066
+L +5V #PWR048
 U 1 1 53F96268
 P 7150 3400
-F 0 "#PWR066" H 7150 3490 20  0001 C CNN
+F 0 "#PWR048" H 7150 3490 20  0001 C CNN
 F 1 "+5V" H 7150 3490 30  0000 C CNN
 F 2 "" H 7150 3400 60  0000 C CNN
@@
 Connection ~ 4150 4200
 $Comp
-L GND #PWR067
+L GND #PWR049
 U 1 1 53FA2AE8
-P 4650 4800
-F 0 "#PWR067" H 4650 4800 30  0001 C CNN
-F 1 "GND" H 4650 4730 30  0001 C CNN
-F 2 "" H 4650 4800 60  0000 C CNN
-F 3 "" H 4650 4800 60  0000 C CNN
-	1    4650 4800
-	1    0    0    -1
-$EndComp
-Wire Wire Line
-	4650 4700 4650 4800
-Wire Wire Line
-	4650 4200 4650 4300
-Connection ~ 4650 4200
-Wire Wire Line
-	4600 4200 5650 4200
+P 4750 5750
+F 0 "#PWR049" H 4750 5750 30  0001 C CNN
+F 1 "GND" H 4750 5680 30  0001 C CNN
+F 2 "" H 4750 5750 60  0000 C CNN
+F 3 "" H 4750 5750 60  0000 C CNN
+	1    4750 5750
+	1    0    0    -1
+$EndComp
+Wire Wire Line
+	4750 5650 4750 5750
 $Comp
 L C C18
@@
 $EndComp
 $Comp
-L GND #PWR068
+L GND #PWR050
 U 1 1 53FF68F8
 P 6850 4000
-F 0 "#PWR068" H 6850 4000 30  0001 C CNN
+F 0 "#PWR050" H 6850 4000 30  0001 C CNN
 F 1 "GND" H 6850 3930 30  0001 C CNN
 F 2 "" H 6850 4000 60  0000 C CNN
@@
 	6850 3500 6700 3500
 Connection ~ 6700 3500
+Text GLabel 4050 3550 0    60   Input ~ 0
+5V_L
+Wire Wire Line
+	4050 3550 4150 3550
+Wire Wire Line
+	4150 3550 4150 3600
+Text GLabel 4700 3950 1    60   Input ~ 0
+CLK_PW_H
+Text GLabel 4750 5200 1    60   Input ~ 0
+CLK_PW_L
+Wire Wire Line
+	4750 5250 4750 5200
+Wire Wire Line
+	4600 4200 5650 4200
+Wire Wire Line
+	4700 4200 4700 3950
+Connection ~ 4700 4200
 $EndSCHEMATC
