File: files/pcb/kicad/USB.sch (KiCad schematic (older format))
At the start: 0 parts

Commit message: 回路図更新
温度湿度センサ
大気圧センサ
輝度センサ
Parts:
- added CON?: USB-MINI-B, ~, symbol USB-MINI-B
- added D? (x2): DIODE, ~, symbol DIODE
- added R? (x2): 68, ~, symbol R
- added R?: NC, ~, symbol R
- added R?: 2K, ~, symbol R
Connections:
- net labels added: +5V, D+, D-, GND
- wire segments 0 -> 24
Changed lines of the file:
@@
 $Descr A4 11693 8268
 encoding utf-8
-Sheet 1 12
+Sheet 5 12
 Title ""
 Date "23 aug 2014"
@@
 Comment4 ""
 $EndDescr
+$Comp
+L USB-MINI-B CON?
+U 1 1 53F90F2D
+P 6150 4200
+F 0 "CON?" H 5900 4650 60  0000 C CNN
+F 1 "USB-MINI-B" H 6100 3700 60  0000 C CNN
+F 2 "~" H 6150 4200 60  0000 C CNN
+F 3 "~" H 6150 4200 60  0000 C CNN
+	1    6150 4200
+	1    0    0    -1
+$EndComp
+Text HLabel 4550 4200 0    60   Input ~ 0
+D+
+Text HLabel 4550 4050 0    60   Input ~ 0
+D-
+$Comp
+L R R?
+U 1 1 53F90F3C
+P 4950 4050
+F 0 "R?" V 5030 4050 40  0000 C CNN
+F 1 "68" V 4957 4051 40  0000 C CNN
+F 2 "~" V 4880 4050 30  0000 C CNN
+F 3 "~" H 4950 4050 30  0000 C CNN
+	1    4950 4050
+	0    -1   -1   0
+$EndComp
+$Comp
+L R R?
+U 1 1 53F90F4B
+P 4950 4200
+F 0 "R?" V 5030 4200 40  0000 C CNN
+F 1 "68" V 4957 4201 40  0000 C CNN
+F 2 "~" V 4880 4200 30  0000 C CNN
+F 3 "~" H 4950 4200 30  0000 C CNN
+	1    4950 4200
+	0    -1   -1   0
+$EndComp
+$Comp
+L GND #PWR?
+U 1 1 53F90F80
+P 6950 5050
+F 0 "#PWR?" H 6950 5050 30  0001 C CNN
+F 1 "GND" H 6950 4980 30  0001 C CNN
+F 2 "" H 6950 5050 60  0000 C CNN
+F 3 "" H 6950 5050 60  0000 C CNN
+	1    6950 5050
+	1    0    0    -1
+$EndComp
+$Comp
+L +5V #PWR?
+U 1 1 53F90F9E
+P 5500 2950
+F 0 "#PWR?" H 5500 3040 20  0001 C CNN
+F 1 "+5V" H 5500 3040 30  0000 C CNN
+F 2 "" H 5500 2950 60  0000 C CNN
+F 3 "" H 5500 2950 60  0000 C CNN
+	1    5500 2950
+	1    0    0    -1
+$EndComp
+$Comp
+L R R?
+U 1 1 53F90FB6
+P 5300 4750
+F 0 "R?" V 5380 4750 40  0000 C CNN
+F 1 "NC" V 5307 4751 40  0000 C CNN
+F 2 "~" V 5230 4750 30  0000 C CNN
+F 3 "~" H 5300 4750 30  0000 C CNN
+	1    5300 4750
+	-1   0    0    1
+$EndComp
+Wire Wire Line
+	6700 3900 6950 3900
+Wire Wire Line
+	6950 3900 6950 4050
+Wire Wire Line
+	6950 4050 6950 4350
+Wire Wire Line
+	6950 4350 6950 4500
+Wire Wire Line
+	6950 4500 6950 5050
+Wire Wire Line
+	6700 4050 6950 4050
+Connection ~ 6950 4050
+Wire Wire Line
+	6700 4350 6950 4350
+Connection ~ 6950 4350
+Wire Wire Line
+	6700 4500 6950 4500
+Connection ~ 6950 4500
+Wire Wire Line
+	5600 3900 5500 3900
+Wire Wire Line
+	5200 4050 5300 4050
+Wire Wire Line
+	5300 4050 5600 4050
+Wire Wire Line
+	5200 4200 5600 4200
+Wire Wire Line
+	4550 4050 4700 4050
+Wire Wire Line
+	4700 4200 4550 4200
+$Comp
+L R R?
+U 1 1 53F91017
+P 5300 3450
+F 0 "R?" V 5380 3450 40  0000 C CNN
+F 1 "2K" V 5307 3451 40  0000 C CNN
+F 2 "~" V 5230 3450 30  0000 C CNN
+F 3 "~" H 5300 3450 30  0000 C CNN
+	1    5300 3450
+	1    0    0    -1
+$EndComp
+Wire Wire Line
+	5300 3700 5300 4050
+Connection ~ 5300 4050
+$Comp
+L +5V #PWR?
+U 1 1 53F91040
+P 5300 2950
+F 0 "#PWR?" H 5300 3040 20  0001 C CNN
+F 1 "+5V" H 5300 3040 30  0000 C CNN
+F 2 "" H 5300 2950 60  0000 C CNN
+F 3 "" H 5300 2950 60  0000 C CNN
+	1    5300 2950
+	1    0    0    -1
+$EndComp
+Wire Wire Line
+	5300 3200 5300 2950
+Wire Wire Line
+	5600 4500 5500 4500
+Wire Wire Line
+	5500 4500 5500 5050
+Wire Wire Line
+	5600 4350 5300 4350
+Wire Wire Line
+	5300 4350 5300 4500
+$Comp
+L GND #PWR?
+U 1 1 53F910A2
+P 5300 5050
+F 0 "#PWR?" H 5300 5050 30  0001 C CNN
+F 1 "GND" H 5300 4980 30  0001 C CNN
+F 2 "" H 5300 5050 60  0000 C CNN
+F 3 "" H 5300 5050 60  0000 C CNN
+	1    5300 5050
+	1    0    0    -1
+$EndComp
+$Comp
+L GND #PWR?
+U 1 1 53F910B1
+P 5500 5050
+F 0 "#PWR?" H 5500 5050 30  0001 C CNN
+F 1 "GND" H 5500 4980 30  0001 C CNN
+F 2 "" H 5500 5050 60  0000 C CNN
+F 3 "" H 5500 5050 60  0000 C CNN
+	1    5500 5050
+	1    0    0    -1
+$EndComp
+Wire Wire Line
+	5300 5000 5300 5050
+$Comp
+L DIODE D?
+U 1 1 53F910F0
+P 5500 3650
+F 0 "D?" H 5500 3750 40  0000 C CNN
+F 1 "DIODE" H 5500 3550 40  0000 C CNN
+F 2 "~" H 5500 3650 60  0000 C CNN
+F 3 "~" H 5500 3650 60  0000 C CNN
+	1    5500 3650
+	0    -1   -1   0
+$EndComp
+$Comp
+L DIODE D?
+U 1 1 53F91104
+P 5500 3200
+F 0 "D?" H 5500 3300 40  0000 C CNN
+F 1 "DIODE" H 5500 3100 40  0000 C CNN
+F 2 "~" H 5500 3200 60  0000 C CNN
+F 3 "~" H 5500 3200 60  0000 C CNN
+	1    5500 3200
+	0    -1   -1   0
+$EndComp
+Wire Wire Line
+	5500 3450 5500 3400
+Wire Wire Line
+	5500 3900 5500 3850
+Wire Wire Line
+	5500 3000 5500 2950
 $EndSCHEMATC

Commit message: 回路図更新、DS1307対応
バスの接続が未
Parts:
- gave numbers to parts that had none: 7
Changed lines of the file:
@@
 $Descr A4 11693 8268
 encoding utf-8
-Sheet 5 12
+Sheet 5 13
 Title ""
-Date "23 aug 2014"
+Date "24 aug 2014"
 Rev ""
 Comp ""
@@
 $EndDescr
 $Comp
-L USB-MINI-B CON?
+L USB-MINI-B CON1
 U 1 1 53F90F2D
 P 6150 4200
-F 0 "CON?" H 5900 4650 60  0000 C CNN
+F 0 "CON1" H 5900 4650 60  0000 C CNN
 F 1 "USB-MINI-B" H 6100 3700 60  0000 C CNN
 F 2 "~" H 6150 4200 60  0000 C CNN
@@
 D-
 $Comp
-L R R?
+L R R16
 U 1 1 53F90F3C
 P 4950 4050
-F 0 "R?" V 5030 4050 40  0000 C CNN
+F 0 "R16" V 5030 4050 40  0000 C CNN
 F 1 "68" V 4957 4051 40  0000 C CNN
 F 2 "~" V 4880 4050 30  0000 C CNN
@@
 $EndComp
 $Comp
-L R R?
+L R R17
 U 1 1 53F90F4B
 P 4950 4200
-F 0 "R?" V 5030 4200 40  0000 C CNN
+F 0 "R17" V 5030 4200 40  0000 C CNN
 F 1 "68" V 4957 4201 40  0000 C CNN
 F 2 "~" V 4880 4200 30  0000 C CNN
@@
 $EndComp
 $Comp
-L GND #PWR?
+L GND #PWR43
 U 1 1 53F90F80
 P 6950 5050
-F 0 "#PWR?" H 6950 5050 30  0001 C CNN
+F 0 "#PWR43" H 6950 5050 30  0001 C CNN
 F 1 "GND" H 6950 4980 30  0001 C CNN
 F 2 "" H 6950 5050 60  0000 C CNN
@@
 $EndComp
 $Comp
-L +5V #PWR?
+L +5V #PWR41
 U 1 1 53F90F9E
 P 5500 2950
-F 0 "#PWR?" H 5500 3040 20  0001 C CNN
+F 0 "#PWR41" H 5500 3040 20  0001 C CNN
 F 1 "+5V" H 5500 3040 30  0000 C CNN
 F 2 "" H 5500 2950 60  0000 C CNN
@@
 $EndComp
 $Comp
-L R R?
+L R R19
 U 1 1 53F90FB6
 P 5300 4750
-F 0 "R?" V 5380 4750 40  0000 C CNN
+F 0 "R19" V 5380 4750 40  0000 C CNN
 F 1 "NC" V 5307 4751 40  0000 C CNN
 F 2 "~" V 5230 4750 30  0000 C CNN
@@
 	4700 4200 4550 4200
 $Comp
-L R R?
+L R R18
 U 1 1 53F91017
 P 5300 3450
-F 0 "R?" V 5380 3450 40  0000 C CNN
+F 0 "R18" V 5380 3450 40  0000 C CNN
 F 1 "2K" V 5307 3451 40  0000 C CNN
 F 2 "~" V 5230 3450 30  0000 C CNN
@@
 Connection ~ 5300 4050
 $Comp
-L +5V #PWR?
+L +5V #PWR39
 U 1 1 53F91040
 P 5300 2950
-F 0 "#PWR?" H 5300 3040 20  0001 C CNN
+F 0 "#PWR39" H 5300 3040 20  0001 C CNN
 F 1 "+5V" H 5300 3040 30  0000 C CNN
 F 2 "" H 5300 2950 60  0000 C CNN
@@
 	5300 4350 5300 4500
 $Comp
-L GND #PWR?
+L GND #PWR40
 U 1 1 53F910A2
 P 5300 5050
-F 0 "#PWR?" H 5300 5050 30  0001 C CNN
+F 0 "#PWR40" H 5300 5050 30  0001 C CNN
 F 1 "GND" H 5300 4980 30  0001 C CNN
 F 2 "" H 5300 5050 60  0000 C CNN
@@
 $EndComp
 $Comp
-L GND #PWR?
+L GND #PWR42
 U 1 1 53F910B1
 P 5500 5050
-F 0 "#PWR?" H 5500 5050 30  0001 C CNN
+F 0 "#PWR42" H 5500 5050 30  0001 C CNN
 F 1 "GND" H 5500 4980 30  0001 C CNN
 F 2 "" H 5500 5050 60  0000 C CNN
@@
 	5300 5000 5300 5050
 $Comp
-L DIODE D?
+L DIODE D5
 U 1 1 53F910F0
 P 5500 3650
-F 0 "D?" H 5500 3750 40  0000 C CNN
+F 0 "D5" H 5500 3750 40  0000 C CNN
 F 1 "DIODE" H 5500 3550 40  0000 C CNN
 F 2 "~" H 5500 3650 60  0000 C CNN
@@
 $EndComp
 $Comp
-L DIODE D?
+L DIODE D4
 U 1 1 53F91104
 P 5500 3200
-F 0 "D?" H 5500 3300 40  0000 C CNN
+F 0 "D4" H 5500 3300 40  0000 C CNN
 F 1 "DIODE" H 5500 3100 40  0000 C CNN
 F 2 "~" H 5500 3200 60  0000 C CNN

Commit message: 回路図ERC途中
Connections:
- wire segments 24 -> 20
Other:
- moved on the sheet: R16, R17, R18
Changed lines of the file:
@@
 $Descr A4 11693 8268
 encoding utf-8
-Sheet 5 13
+Sheet 6 13
 Title ""
-Date "24 aug 2014"
+Date "25 aug 2014"
 Rev ""
 Comp ""
@@
 Comment4 ""
 $EndDescr
-$Comp
-L USB-MINI-B CON1
-U 1 1 53F90F2D
-P 6150 4200
-F 0 "CON1" H 5900 4650 60  0000 C CNN
-F 1 "USB-MINI-B" H 6100 3700 60  0000 C CNN
-F 2 "~" H 6150 4200 60  0000 C CNN
-F 3 "~" H 6150 4200 60  0000 C CNN
-	1    6150 4200
-	1    0    0    -1
-$EndComp
-Text HLabel 4550 4200 0    60   Input ~ 0
+Text HLabel 4400 4200 0    60   Input ~ 0
 D+
-Text HLabel 4550 4050 0    60   Input ~ 0
+Text HLabel 4400 4050 0    60   Input ~ 0
 D-
 $Comp
 L R R16
 U 1 1 53F90F3C
-P 4950 4050
-F 0 "R16" V 5030 4050 40  0000 C CNN
-F 1 "68" V 4957 4051 40  0000 C CNN
-F 2 "~" V 4880 4050 30  0000 C CNN
-F 3 "~" H 4950 4050 30  0000 C CNN
-	1    4950 4050
+P 4800 4050
+F 0 "R16" V 4880 4050 40  0000 C CNN
+F 1 "68" V 4807 4051 40  0000 C CNN
+F 2 "~" V 4730 4050 30  0000 C CNN
+F 3 "~" H 4800 4050 30  0000 C CNN
+	1    4800 4050
 	0    -1   -1   0
 $EndComp
@@
 L R R17
 U 1 1 53F90F4B
-P 4950 4200
-F 0 "R17" V 5030 4200 40  0000 C CNN
-F 1 "68" V 4957 4201 40  0000 C CNN
-F 2 "~" V 4880 4200 30  0000 C CNN
-F 3 "~" H 4950 4200 30  0000 C CNN
-	1    4950 4200
+P 4800 4200
+F 0 "R17" V 4880 4200 40  0000 C CNN
+F 1 "68" V 4807 4201 40  0000 C CNN
+F 2 "~" V 4730 4200 30  0000 C CNN
+F 3 "~" H 4800 4200 30  0000 C CNN
+	1    4800 4200
 	0    -1   -1   0
 $EndComp
 $Comp
-L GND #PWR43
+L GND #PWR039
 U 1 1 53F90F80
 P 6950 5050
-F 0 "#PWR43" H 6950 5050 30  0001 C CNN
+F 0 "#PWR039" H 6950 5050 30  0001 C CNN
 F 1 "GND" H 6950 4980 30  0001 C CNN
 F 2 "" H 6950 5050 60  0000 C CNN
@@
 $EndComp
 $Comp
-L +5V #PWR41
+L +5V #PWR040
 U 1 1 53F90F9E
 P 5500 2950
-F 0 "#PWR41" H 5500 3040 20  0001 C CNN
+F 0 "#PWR040" H 5500 3040 20  0001 C CNN
 F 1 "+5V" H 5500 3040 30  0000 C CNN
 F 2 "" H 5500 2950 60  0000 C CNN
@@
 	6700 3900 6950 3900
 Wire Wire Line
-	6950 3900 6950 4050
-Wire Wire Line
-	6950 4050 6950 4350
-Wire Wire Line
-	6950 4350 6950 4500
-Wire Wire Line
-	6950 4500 6950 5050
+	6950 3900 6950 5050
 Wire Wire Line
 	6700 4050 6950 4050
@@
 Connection ~ 6950 4500
 Wire Wire Line
-	5600 3900 5500 3900
+	5050 4050 5600 4050
 Wire Wire Line
-	5200 4050 5300 4050
+	5050 4200 5600 4200
 Wire Wire Line
-	5300 4050 5600 4050
+	4400 4050 4550 4050
 Wire Wire Line
-	5200 4200 5600 4200
-Wire Wire Line
-	4550 4050 4700 4050
-Wire Wire Line
-	4700 4200 4550 4200
+	4550 4200 4400 4200
 $Comp
 L R R18
 U 1 1 53F91017
-P 5300 3450
-F 0 "R18" V 5380 3450 40  0000 C CNN
-F 1 "2K" V 5307 3451 40  0000 C CNN
-F 2 "~" V 5230 3450 30  0000 C CNN
-F 3 "~" H 5300 3450 30  0000 C CNN
-	1    5300 3450
+P 5150 3450
+F 0 "R18" V 5230 3450 40  0000 C CNN
+F 1 "2K" V 5157 3451 40  0000 C CNN
+F 2 "~" V 5080 3450 30  0000 C CNN
+F 3 "~" H 5150 3450 30  0000 C CNN
+	1    5150 3450
 	1    0    0    -1
 $EndComp
 Wire Wire Line
-	5300 3700 5300 4050
-Connection ~ 5300 4050
+	5150 3700 5150 4050
+Connection ~ 5150 4050
 $Comp
-L +5V #PWR39
+L +5V #PWR041
 U 1 1 53F91040
-P 5300 2950
-F 0 "#PWR39" H 5300 3040 20  0001 C CNN
-F 1 "+5V" H 5300 3040 30  0000 C CNN
-F 2 "" H 5300 2950 60  0000 C CNN
-F 3 "" H 5300 2950 60  0000 C CNN
-	1    5300 2950
+P 5150 2950
+F 0 "#PWR041" H 5150 3040 20  0001 C CNN
+F 1 "+5V" H 5150 3040 30  0000 C CNN
+F 2 "" H 5150 2950 60  0000 C CNN
+F 3 "" H 5150 2950 60  0000 C CNN
+	1    5150 2950
 	1    0    0    -1
 $EndComp
 Wire Wire Line
-	5300 3200 5300 2950
+	5150 3200 5150 2950
 Wire Wire Line
 	5600 4500 5500 4500
@@
 	5300 4350 5300 4500
 $Comp
-L GND #PWR40
+L GND #PWR042
 U 1 1 53F910A2
 P 5300 5050
-F 0 "#PWR40" H 5300 5050 30  0001 C CNN
+F 0 "#PWR042" H 5300 5050 30  0001 C CNN
 F 1 "GND" H 5300 4980 30  0001 C CNN
 F 2 "" H 5300 5050 60  0000 C CNN
@@
 $EndComp
 $Comp
-L GND #PWR42
+L GND #PWR043
 U 1 1 53F910B1
 P 5500 5050
-F 0 "#PWR42" H 5500 5050 30  0001 C CNN
+F 0 "#PWR043" H 5500 5050 30  0001 C CNN
 F 1 "GND" H 5500 4980 30  0001 C CNN
 F 2 "" H 5500 5050 60  0000 C CNN
@@
 Wire Wire Line
 	5500 3000 5500 2950
+$Comp
+L USB-MINI-B CON1
+U 1 1 53F90F2D
+P 6150 4200
+F 0 "CON1" H 5900 4650 60  0000 C CNN
+F 1 "USB-MINI-B" H 6100 3700 60  0000 C CNN
+F 2 "~" H 6150 4200 60  0000 C CNN
+F 3 "~" H 6150 4200 60  0000 C CNN
+	1    6150 4200
+	1    0    0    -1
+$EndComp
+Wire Wire Line
+	5600 3900 5500 3900
 $EndSCHEMATC

Commit message: 回路図ERC完了
Parts:
- removed CON1: USB-MINI-B, ~, symbol USB-MINI-B
- added CON1: USB_MINI_B, ~, symbol USB_MINI_B
Connections:
- wire segments 20 -> 21
Other:
- moved on the sheet: D4, D5, R16, R17, R18, R19
Changed lines of the file:
@@
 Sheet 6 13
 Title ""
-Date "25 aug 2014"
+Date "26 aug 2014"
 Rev ""
 Comp ""
@@
 Comment4 ""
 $EndDescr
-Text HLabel 4400 4200 0    60   Input ~ 0
+Text HLabel 4200 4200 0    60   Input ~ 0
 D+
-Text HLabel 4400 4050 0    60   Input ~ 0
+Text HLabel 4200 4050 0    60   Input ~ 0
 D-
 $Comp
 L R R16
 U 1 1 53F90F3C
-P 4800 4050
-F 0 "R16" V 4880 4050 40  0000 C CNN
-F 1 "68" V 4807 4051 40  0000 C CNN
-F 2 "~" V 4730 4050 30  0000 C CNN
-F 3 "~" H 4800 4050 30  0000 C CNN
-	1    4800 4050
+P 4600 4050
+F 0 "R16" V 4680 4050 40  0000 C CNN
+F 1 "68" V 4607 4051 40  0000 C CNN
+F 2 "~" V 4530 4050 30  0000 C CNN
+F 3 "~" H 4600 4050 30  0000 C CNN
+	1    4600 4050
 	0    -1   -1   0
 $EndComp
@@
 L R R17
 U 1 1 53F90F4B
-P 4800 4200
-F 0 "R17" V 4880 4200 40  0000 C CNN
-F 1 "68" V 4807 4201 40  0000 C CNN
-F 2 "~" V 4730 4200 30  0000 C CNN
-F 3 "~" H 4800 4200 30  0000 C CNN
-	1    4800 4200
-	0    -1   -1   0
-$EndComp
-$Comp
-L GND #PWR039
-U 1 1 53F90F80
-P 6950 5050
-F 0 "#PWR039" H 6950 5050 30  0001 C CNN
-F 1 "GND" H 6950 4980 30  0001 C CNN
-F 2 "" H 6950 5050 60  0000 C CNN
-F 3 "" H 6950 5050 60  0000 C CNN
-	1    6950 5050
-	1    0    0    -1
-$EndComp
-$Comp
-L +5V #PWR040
+P 4600 4200
+F 0 "R17" V 4680 4200 40  0000 C CNN
+F 1 "68" V 4607 4201 40  0000 C CNN
+F 2 "~" V 4530 4200 30  0000 C CNN
+F 3 "~" H 4600 4200 30  0000 C CNN
+	1    4600 4200
+	0    -1   -1   0
+$EndComp
+$Comp
+L +5V #PWR046
 U 1 1 53F90F9E
-P 5500 2950
-F 0 "#PWR040" H 5500 3040 20  0001 C CNN
-F 1 "+5V" H 5500 3040 30  0000 C CNN
-F 2 "" H 5500 2950 60  0000 C CNN
-F 3 "" H 5500 2950 60  0000 C CNN
-	1    5500 2950
+P 5300 2950
+F 0 "#PWR046" H 5300 3040 20  0001 C CNN
+F 1 "+5V" H 5300 3040 30  0000 C CNN
+F 2 "" H 5300 2950 60  0000 C CNN
+F 3 "" H 5300 2950 60  0000 C CNN
+	1    5300 2950
 	1    0    0    -1
 $EndComp
@@
 L R R19
 U 1 1 53F90FB6
-P 5300 4750
-F 0 "R19" V 5380 4750 40  0000 C CNN
-F 1 "NC" V 5307 4751 40  0000 C CNN
-F 2 "~" V 5230 4750 30  0000 C CNN
-F 3 "~" H 5300 4750 30  0000 C CNN
-	1    5300 4750
+P 5100 4750
+F 0 "R19" V 5180 4750 40  0000 C CNN
+F 1 "NC" V 5107 4751 40  0000 C CNN
+F 2 "~" V 5030 4750 30  0000 C CNN
+F 3 "~" H 5100 4750 30  0000 C CNN
+	1    5100 4750
 	-1   0    0    1
 $EndComp
-Wire Wire Line
-	6700 3900 6950 3900
-Wire Wire Line
-	6950 3900 6950 5050
-Wire Wire Line
-	6700 4050 6950 4050
-Connection ~ 6950 4050
-Wire Wire Line
-	6700 4350 6950 4350
-Connection ~ 6950 4350
-Wire Wire Line
-	6700 4500 6950 4500
-Connection ~ 6950 4500
-Wire Wire Line
-	5050 4050 5600 4050
-Wire Wire Line
-	5050 4200 5600 4200
-Wire Wire Line
-	4400 4050 4550 4050
-Wire Wire Line
-	4550 4200 4400 4200
 $Comp
 L R R18
 U 1 1 53F91017
-P 5150 3450
-F 0 "R18" V 5230 3450 40  0000 C CNN
-F 1 "2K" V 5157 3451 40  0000 C CNN
-F 2 "~" V 5080 3450 30  0000 C CNN
-F 3 "~" H 5150 3450 30  0000 C CNN
-	1    5150 3450
-	1    0    0    -1
-$EndComp
-Wire Wire Line
-	5150 3700 5150 4050
-Connection ~ 5150 4050
-$Comp
-L +5V #PWR041
+P 4950 3450
+F 0 "R18" V 5030 3450 40  0000 C CNN
+F 1 "2K" V 4957 3451 40  0000 C CNN
+F 2 "~" V 4880 3450 30  0000 C CNN
+F 3 "~" H 4950 3450 30  0000 C CNN
+	1    4950 3450
+	1    0    0    -1
+$EndComp
+$Comp
+L +5V #PWR047
 U 1 1 53F91040
-P 5150 2950
-F 0 "#PWR041" H 5150 3040 20  0001 C CNN
-F 1 "+5V" H 5150 3040 30  0000 C CNN
-F 2 "" H 5150 2950 60  0000 C CNN
-F 3 "" H 5150 2950 60  0000 C CNN
-	1    5150 2950
-	1    0    0    -1
-$EndComp
-Wire Wire Line
-	5150 3200 5150 2950
-Wire Wire Line
-	5600 4500 5500 4500
-Wire Wire Line
-	5500 4500 5500 5050
-Wire Wire Line
-	5600 4350 5300 4350
-Wire Wire Line
-	5300 4350 5300 4500
-$Comp
-L GND #PWR042
+P 4950 2950
+F 0 "#PWR047" H 4950 3040 20  0001 C CNN
+F 1 "+5V" H 4950 3040 30  0000 C CNN
+F 2 "" H 4950 2950 60  0000 C CNN
+F 3 "" H 4950 2950 60  0000 C CNN
+	1    4950 2950
+	1    0    0    -1
+$EndComp
+$Comp
+L GND #PWR048
 U 1 1 53F910A2
+P 5100 5050
+F 0 "#PWR048" H 5100 5050 30  0001 C CNN
+F 1 "GND" H 5100 4980 30  0001 C CNN
+F 2 "" H 5100 5050 60  0000 C CNN
+F 3 "" H 5100 5050 60  0000 C CNN
+	1    5100 5050
+	1    0    0    -1
+$EndComp
+$Comp
+L GND #PWR049
+U 1 1 53F910B1
 P 5300 5050
-F 0 "#PWR042" H 5300 5050 30  0001 C CNN
+F 0 "#PWR049" H 5300 5050 30  0001 C CNN
 F 1 "GND" H 5300 4980 30  0001 C CNN
 F 2 "" H 5300 5050 60  0000 C CNN
@@
 $EndComp
 $Comp
-L GND #PWR043
-U 1 1 53F910B1
-P 5500 5050
-F 0 "#PWR043" H 5500 5050 30  0001 C CNN
-F 1 "GND" H 5500 4980 30  0001 C CNN
-F 2 "" H 5500 5050 60  0000 C CNN
-F 3 "" H 5500 5050 60  0000 C CNN
-	1    5500 5050
-	1    0    0    -1
-$EndComp
-Wire Wire Line
-	5300 5000 5300 5050
-$Comp
 L DIODE D5
 U 1 1 53F910F0
-P 5500 3650
-F 0 "D5" H 5500 3750 40  0000 C CNN
-F 1 "DIODE" H 5500 3550 40  0000 C CNN
-F 2 "~" H 5500 3650 60  0000 C CNN
-F 3 "~" H 5500 3650 60  0000 C CNN
-	1    5500 3650
+P 5300 3650
+F 0 "D5" H 5300 3750 40  0000 C CNN
+F 1 "DIODE" H 5300 3550 40  0000 C CNN
+F 2 "~" H 5300 3650 60  0000 C CNN
+F 3 "~" H 5300 3650 60  0000 C CNN
+	1    5300 3650
 	0    -1   -1   0
 $EndComp
@@
 L DIODE D4
 U 1 1 53F91104
-P 5500 3200
-F 0 "D4" H 5500 3300 40  0000 C CNN
-F 1 "DIODE" H 5500 3100 40  0000 C CNN
-F 2 "~" H 5500 3200 60  0000 C CNN
-F 3 "~" H 5500 3200 60  0000 C CNN
-	1    5500 3200
-	0    -1   -1   0
-$EndComp
-Wire Wire Line
-	5500 3450 5500 3400
-Wire Wire Line
-	5500 3900 5500 3850
-Wire Wire Line
-	5500 3000 5500 2950
-$Comp
-L USB-MINI-B CON1
-U 1 1 53F90F2D
+P 5300 3200
+F 0 "D4" H 5300 3300 40  0000 C CNN
+F 1 "DIODE" H 5300 3100 40  0000 C CNN
+F 2 "~" H 5300 3200 60  0000 C CNN
+F 3 "~" H 5300 3200 60  0000 C CNN
+	1    5300 3200
+	0    -1   -1   0
+$EndComp
+$Comp
+L PWR_FLAG #FLG050
+U 1 1 53FCAA4C
+P 5550 3800
+F 0 "#FLG050" H 5550 3895 30  0001 C CNN
+F 1 "PWR_FLAG" H 5550 3980 30  0000 C CNN
+F 2 "" H 5550 3800 60  0000 C CNN
+F 3 "" H 5550 3800 60  0000 C CNN
+	1    5550 3800
+	1    0    0    -1
+$EndComp
+$Comp
+L GND #PWR051
+U 1 1 53FCBB40
+P 6950 4600
+F 0 "#PWR051" H 6950 4600 30  0001 C CNN
+F 1 "GND" H 6950 4530 30  0001 C CNN
+F 2 "" H 6950 4600 60  0000 C CNN
+F 3 "" H 6950 4600 60  0000 C CNN
+	1    6950 4600
+	1    0    0    -1
+$EndComp
+Wire Wire Line
+	4850 4050 5600 4050
+Wire Wire Line
+	4850 4200 5600 4200
+Wire Wire Line
+	4200 4050 4350 4050
+Wire Wire Line
+	4350 4200 4200 4200
+Wire Wire Line
+	4950 3700 4950 4050
+Connection ~ 4950 4050
+Wire Wire Line
+	4950 3200 4950 2950
+Wire Wire Line
+	5600 4500 5300 4500
+Wire Wire Line
+	5300 4500 5300 5050
+Wire Wire Line
+	5600 4350 5100 4350
+Wire Wire Line
+	5100 4350 5100 4500
+Wire Wire Line
+	5100 5000 5100 5050
+Wire Wire Line
+	5300 3450 5300 3400
+Wire Wire Line
+	5300 3900 5300 3850
+Wire Wire Line
+	5300 3000 5300 2950
+Wire Wire Line
+	5600 3900 5300 3900
+Wire Wire Line
+	5550 3800 5550 3900
+Connection ~ 5550 3900
+Wire Wire Line
+	6700 3900 6950 3900
+Wire Wire Line
+	6950 3900 6950 4600
+Wire Wire Line
+	6700 4050 6950 4050
+Connection ~ 6950 4050
+Wire Wire Line
+	6700 4350 6950 4350
+Connection ~ 6950 4350
+Wire Wire Line
+	6700 4500 6950 4500
+Connection ~ 6950 4500
+$Comp
+L USB_MINI_B CON1
+U 1 1 53FCC671
 P 6150 4200
 F 0 "CON1" H 5900 4650 60  0000 C CNN
-F 1 "USB-MINI-B" H 6100 3700 60  0000 C CNN
+F 1 "USB_MINI_B" H 6100 3700 60  0000 C CNN
 F 2 "~" H 6150 4200 60  0000 C CNN
 F 3 "~" H 6150 4200 60  0000 C CNN
@@
 	1    0    0    -1
 $EndComp
-Wire Wire Line
-	5600 3900 5500 3900
 $EndSCHEMATC

Commit message: 部品リスト・パッケージライブラリを更新
Parts:
- renumbered D4 to D3, D5 to D4, R16 to R20, R17 to R21, R18 to R22, R19 to R23
Changed lines of the file:
@@
 D-
 $Comp
-L R R16
+L R R20
 U 1 1 53F90F3C
 P 4600 4050
-F 0 "R16" V 4680 4050 40  0000 C CNN
+F 0 "R20" V 4680 4050 40  0000 C CNN
 F 1 "68" V 4607 4051 40  0000 C CNN
 F 2 "~" V 4530 4050 30  0000 C CNN
@@
 $EndComp
 $Comp
-L R R17
+L R R21
 U 1 1 53F90F4B
 P 4600 4200
-F 0 "R17" V 4680 4200 40  0000 C CNN
+F 0 "R21" V 4680 4200 40  0000 C CNN
 F 1 "68" V 4607 4201 40  0000 C CNN
 F 2 "~" V 4530 4200 30  0000 C CNN
@@
 $EndComp
 $Comp
-L R R19
+L R R23
 U 1 1 53F90FB6
 P 5100 4750
-F 0 "R19" V 5180 4750 40  0000 C CNN
+F 0 "R23" V 5180 4750 40  0000 C CNN
 F 1 "NC" V 5107 4751 40  0000 C CNN
 F 2 "~" V 5030 4750 30  0000 C CNN
@@
 $EndComp
 $Comp
-L R R18
+L R R22
 U 1 1 53F91017
 P 4950 3450
-F 0 "R18" V 5030 3450 40  0000 C CNN
+F 0 "R22" V 5030 3450 40  0000 C CNN
 F 1 "2K" V 4957 3451 40  0000 C CNN
 F 2 "~" V 4880 3450 30  0000 C CNN
@@
 $EndComp
 $Comp
-L DIODE D5
+L DIODE D4
 U 1 1 53F910F0
 P 5300 3650
-F 0 "D5" H 5300 3750 40  0000 C CNN
+F 0 "D4" H 5300 3750 40  0000 C CNN
 F 1 "DIODE" H 5300 3550 40  0000 C CNN
 F 2 "~" H 5300 3650 60  0000 C CNN
@@
 $EndComp
 $Comp
-L DIODE D4
+L DIODE D3
 U 1 1 53F91104
 P 5300 3200
-F 0 "D4" H 5300 3300 40  0000 C CNN
+F 0 "D3" H 5300 3300 40  0000 C CNN
 F 1 "DIODE" H 5300 3100 40  0000 C CNN
 F 2 "~" H 5300 3200 60  0000 C CNN
