File: files/pcb/kicad/kicad_project.sch (KiCad schematic (older format))
At the start: 2 parts, among them IC1 ICM7555CD, IC2 ICM7555CD

Commit message: 回路更新
マイコン周り作成、各子階層シートを追加
Parts:
- removed IC1, IC2: ICM7555CD, ~, symbol ICM7555CD
- added C? (x4): C, ~, symbol C
- added D?: LED, ~, symbol LED
- added D?: DIODE, ~, symbol DIODE
- added IC?: ATMEGA328-A, TQFP32, symbol ATMEGA328-A
- added R? (x5): R, ~, symbol R
- added R?: 10k, ~, symbol R
- added SW?: SW_PUSH, ~, symbol SW_PUSH
- added X?: CRYSTAL, ~, symbol CRYSTAL
Connections:
- wire segments 9 -> 100
- no-connect marks 0 -> 1

Commit message: 回路図更新、DS1307対応
バスの接続が未
Parts:
- removed D?: LED, ~, symbol LED
- removed R?: R, ~, symbol R
- gave numbers to parts that had none: 13
Connections:
- wire segments 100 -> 92
- no-connect marks 1 -> 2
Other:
- moved on the sheet: R4, R5

Commit message: 回路図ERC途中
Parts:
- added C13: 0.1u, ~, symbol C
- C1: value C -> 0.1u
- C2: value C -> 10u
- C3, C4: value C -> 22p
- R2: value R -> 1k
Connections:
- net +5V: now also C13.1
- net GND: now also C13.2
- net Sheet53F9209A/out: now also IC1.31 ((PCINT17/TXD)PD1)
- net PB0: now reaches IC1.12 ((PCINT0/CLKO/ICP1)PB0)
- net PB1: now reaches IC1.13 ((PCINT1/OC1A)PB1)
- net PB2: now reaches IC1.14 ((PCINT2/OC1B/~SS~)PB2)
- net PB3: now reaches IC1.15 ((PCINT3/OC2A/MOSI)PB3)
- net PB4: now reaches IC1.16 ((PCINT4/MISO)PB4)
- net PC0: now reaches IC1.23 ((PCINT8/ADC0)PC0)
- net PC1: now reaches IC1.24 ((PCINT9/ADC1)PC1)
- net PC2: now reaches IC1.25 ((PCINT10/ADC2)PC2)
- net PC3: now reaches IC1.26 ((PCINT11/ADC3)PC3)
Other:
- moved on the sheet: C1, C3, C4, IC1, R1, X1

Commit message: 回路図ERC完了
Parts:
- added P1: CONN_6, ~, symbol CONN_6
Connections:
- net +5V: now also P1.6
- net GND: now also P1.3
- net RESET: now reaches IC1.29 ((PCINT14/~RESET~)PC6), R2.1
- net RESET: now also P1.1
- net PB3 renamed MOSI
- net MOSI: now also P1.5
- net PB4 renamed MISO
- net MISO: now also P1.4
- net Sheet53F91D14/beep renamed SCK
- net SCK: now also P1.2
- no-connect marks 2 -> 1
Other:
- note added: "9V in - 170V out, 5V out"
- note added: "ISP tool (In system programmer)"
- note added: "Reset circuit\nstartup in 0.1[sec]"
- moved on the sheet: C2, D1, R2, R3, SW1
Changed lines of the file:
@@
 Sheet 1 13
 Title ""
-Date "25 aug 2014"
+Date "26 aug 2014"
 Rev ""
 Comp ""
@@
 $EndSheet
 $Sheet
-S 1300 1000 1100 500
+S 1300 1200 1100 500
 U 53F8942B
 F0 "Sheet53F8942A" 50
@@
 L SW_PUSH SW1
 U 1 1 53F90D02
-P 4800 6600
-F 0 "SW1" H 4950 6710 50  0000 C CNN
-F 1 "SW_PUSH" H 4800 6520 50  0000 C CNN
-F 2 "~" H 4800 6600 60  0000 C CNN
-F 3 "~" H 4800 6600 60  0000 C CNN
-	1    4800 6600
+P 4950 6600
+F 0 "SW1" H 5100 6710 50  0000 C CNN
+F 1 "SW_PUSH" H 4950 6520 50  0000 C CNN
+F 2 "~" H 4950 6600 60  0000 C CNN
+F 3 "~" H 4950 6600 60  0000 C CNN
+	1    4950 6600
 	0    -1   1    0
 $EndComp
@@
 L GND #PWR07
 U 1 1 53F90D11
-P 5050 6900
-F 0 "#PWR07" H 5050 6900 30  0001 C CNN
-F 1 "GND" H 5050 6830 30  0001 C CNN
-F 2 "" H 5050 6900 60  0000 C CNN
-F 3 "" H 5050 6900 60  0000 C CNN
-	1    5050 6900
+P 5200 6900
+F 0 "#PWR07" H 5200 6900 30  0001 C CNN
+F 1 "GND" H 5200 6830 30  0001 C CNN
+F 2 "" H 5200 6900 60  0000 C CNN
+F 3 "" H 5200 6900 60  0000 C CNN
+	1    5200 6900
 	-1   0    0    -1
 $EndComp
@@
 L C C2
 U 1 1 53F90D20
-P 5050 6600
-F 0 "C2" H 5050 6700 40  0000 L CNN
-F 1 "10u" H 4900 6500 40  0000 L CNN
-F 2 "~" H 5088 6450 30  0000 C CNN
-F 3 "~" H 5050 6600 60  0000 C CNN
-	1    5050 6600
+P 5200 6600
+F 0 "C2" H 5200 6700 40  0000 L CNN
+F 1 "10u" H 5050 6500 40  0000 L CNN
+F 2 "~" H 5238 6450 30  0000 C CNN
+F 3 "~" H 5200 6600 60  0000 C CNN
+	1    5200 6600
 	-1   0    0    -1
 $EndComp
@@
 L R R3
 U 1 1 53F90D2F
-P 5050 6050
-F 0 "R3" V 5130 6050 40  0000 C CNN
-F 1 "10k" V 5057 6051 40  0000 C CNN
-F 2 "~" V 4980 6050 30  0000 C CNN
-F 3 "~" H 5050 6050 30  0000 C CNN
-	1    5050 6050
+P 5200 6050
+F 0 "R3" V 5280 6050 40  0000 C CNN
+F 1 "10k" V 5207 6051 40  0000 C CNN
+F 2 "~" V 5130 6050 30  0000 C CNN
+F 3 "~" H 5200 6050 30  0000 C CNN
+	1    5200 6050
 	-1   0    0    -1
 $EndComp
@@
 L +5V #PWR08
 U 1 1 53F90D3E
-P 5050 5800
-F 0 "#PWR08" H 5050 5890 20  0001 C CNN
-F 1 "+5V" H 5050 5890 30  0000 C CNN
-F 2 "" H 5050 5800 60  0000 C CNN
-F 3 "" H 5050 5800 60  0000 C CNN
-	1    5050 5800
+P 5200 5800
+F 0 "#PWR08" H 5200 5890 20  0001 C CNN
+F 1 "+5V" H 5200 5890 30  0000 C CNN
+F 2 "" H 5200 5800 60  0000 C CNN
+F 3 "" H 5200 5800 60  0000 C CNN
+	1    5200 5800
 	-1   0    0    -1
 $EndComp
@@
 L GND #PWR09
 U 1 1 53F90DED
-P 4800 6950
-F 0 "#PWR09" H 4800 6950 30  0001 C CNN
-F 1 "GND" H 4800 6880 30  0001 C CNN
-F 2 "" H 4800 6950 60  0000 C CNN
-F 3 "" H 4800 6950 60  0000 C CNN
-	1    4800 6950
+P 4950 6950
+F 0 "#PWR09" H 4950 6950 30  0001 C CNN
+F 1 "GND" H 4950 6880 30  0001 C CNN
+F 2 "" H 4950 6950 60  0000 C CNN
+F 3 "" H 4950 6950 60  0000 C CNN
+	1    4950 6950
 	-1   0    0    -1
 $EndComp
@@
 L DIODE D1
 U 1 1 53F911D9
-P 5300 6050
-F 0 "D1" H 5300 6150 40  0000 C CNN
-F 1 "DIODE" H 5300 5950 40  0000 C CNN
-F 2 "~" H 5300 6050 60  0000 C CNN
-F 3 "~" H 5300 6050 60  0000 C CNN
-	1    5300 6050
+P 5450 6050
+F 0 "D1" H 5450 6150 40  0000 C CNN
+F 1 "DIODE" H 5450 5950 40  0000 C CNN
+F 2 "~" H 5450 6050 60  0000 C CNN
+F 3 "~" H 5450 6050 60  0000 C CNN
+	1    5450 6050
 	0    1    -1   0
 $EndComp
@@
 L +5V #PWR010
 U 1 1 53F911E8
-P 5300 5800
-F 0 "#PWR010" H 5300 5890 20  0001 C CNN
-F 1 "+5V" H 5300 5890 30  0000 C CNN
-F 2 "" H 5300 5800 60  0000 C CNN
-F 3 "" H 5300 5800 60  0000 C CNN
-	1    5300 5800
+P 5450 5800
+F 0 "#PWR010" H 5450 5890 20  0001 C CNN
+F 1 "+5V" H 5450 5890 30  0000 C CNN
+F 2 "" H 5450 5800 60  0000 C CNN
+F 3 "" H 5450 5800 60  0000 C CNN
+	1    5450 5800
 	-1   0    0    -1
 $EndComp
@@
 L R R2
 U 1 1 53F911F7
-P 4800 6050
-F 0 "R2" V 4880 6050 40  0000 C CNN
-F 1 "1k" V 4807 6051 40  0000 C CNN
-F 2 "~" V 4730 6050 30  0000 C CNN
-F 3 "~" H 4800 6050 30  0000 C CNN
-	1    4800 6050
+P 4950 6050
+F 0 "R2" V 5030 6050 40  0000 C CNN
+F 1 "1k" V 4957 6051 40  0000 C CNN
+F 2 "~" V 4880 6050 30  0000 C CNN
+F 3 "~" H 4950 6050 30  0000 C CNN
+	1    4950 6050
 	-1   0    0    -1
 $EndComp
@@
 F1 "RTC_DS1307.sch" 50
 F2 "CLKOUT" I L 7350 3000 60
-F3 "CLKEN" I L 7350 3100 60
-F4 "SDA" I L 7350 2800 60
-F5 "SCL" I L 7350 2900 60
+F3 "SDA" I L 7350 2800 60
+F4 "SCL" I L 7350 2900 60
 $EndSheet
 $Sheet
@@
 F3 "SCL" I L 9550 2900 60
 $EndSheet
-NoConn ~ 7350 3100
 Entry Wire Line
 	4750 3400 4850 3300
@@
 Text Label 4950 1350 0    60   ~ 0
 PB[0..4]
+Text Label 4500 3300 0    60   ~ 0
+PB3
+Text Label 4500 3400 0    60   ~ 0
+PB4
+$Comp
+L CONN_6 P1
+U 1 1 53FCD3BC
+P 3100 1500
+F 0 "P1" V 3050 1500 60  0000 C CNN
+F 1 "CONN_6" V 3150 1500 60  0000 C CNN
+F 2 "~" H 3100 1500 60  0000 C CNN
+F 3 "~" H 3100 1500 60  0000 C CNN
+	1    3100 1500
+	-1   0    0    1
+$EndComp
+Text Label 4500 4450 0    60   ~ 0
+RESET
+Text Label 4500 3500 0    60   ~ 0
+SCK
+Text Label 3550 1750 0    60   ~ 0
+RESET
+Text Label 3550 1650 0    60   ~ 0
+SCK
+Text Label 3550 1450 0    60   ~ 0
+MISO
+Text Label 4700 3400 0    60   ~ 0
+MISO
+Text Label 4700 3300 0    60   ~ 0
+MOSI
+Text Label 3550 1350 0    60   ~ 0
+MOSI
+$Comp
+L +5V #PWR013
+U 1 1 53FCE0E8
+P 3850 1150
+F 0 "#PWR013" H 3850 1240 20  0001 C CNN
+F 1 "+5V" H 3850 1240 30  0000 C CNN
+F 2 "" H 3850 1150 60  0000 C CNN
+F 3 "" H 3850 1150 60  0000 C CNN
+	1    3850 1150
+	1    0    0    -1
+$EndComp
+$Comp
+L GND #PWR014
+U 1 1 53FCE0F7
+P 3850 1900
+F 0 "#PWR014" H 3850 1900 30  0001 C CNN
+F 1 "GND" H 3850 1830 30  0001 C CNN
+F 2 "" H 3850 1900 60  0000 C CNN
+F 3 "" H 3850 1900 60  0000 C CNN
+	1    3850 1900
+	1    0    0    -1
+$EndComp
 Connection ~ 2400 5100
 Connection ~ 2400 3300
@@
 	7150 4600 4450 4600
 Wire Wire Line
-	4450 4450 4800 4450
-Wire Wire Line
-	5050 6300 5050 6400
-Wire Wire Line
-	5050 6800 5050 6900
-Wire Wire Line
-	4800 6300 5300 6300
-Wire Wire Line
-	4800 4450 4800 5800
-Wire Wire Line
-	5300 6300 5300 6250
-Connection ~ 5050 6300
-Connection ~ 4800 6300
-Wire Wire Line
-	5300 5850 5300 5800
+	4450 4450 4950 4450
+Wire Wire Line
+	5200 6300 5200 6400
+Wire Wire Line
+	5200 6800 5200 6900
+Wire Wire Line
+	4950 6300 5450 6300
+Wire Wire Line
+	4950 4450 4950 5800
+Wire Wire Line
+	5450 6300 5450 6250
+Connection ~ 5200 6300
+Connection ~ 4950 6300
+Wire Wire Line
+	5450 5850 5450 5800
 Wire Wire Line
 	5050 5300 5050 5450
@@
 Wire Bus Line
 	4950 1750 5400 1750
-Text Label 4500 3300 0    60   ~ 0
-PB3
-Text Label 4500 3400 0    60   ~ 0
-PB4
 Wire Bus Line
-	4850 3300 4850 1350
+	4850 1350 4850 3300
 Wire Bus Line
-	4950 4050 4950 1750
-Wire Wire Line
-	4800 6900 4800 6950
+	4950 1750 4950 4050
+Wire Wire Line
+	4950 6900 4950 6950
+Wire Wire Line
+	3450 1250 3850 1250
+Wire Wire Line
+	3850 1250 3850 1150
+Wire Wire Line
+	3450 1550 3850 1550
+Wire Wire Line
+	3850 1550 3850 1900
+Wire Wire Line
+	3450 1350 3550 1350
+Wire Wire Line
+	3550 1450 3450 1450
+Wire Wire Line
+	3450 1650 3550 1650
+Wire Wire Line
+	3550 1750 3450 1750
+Text Notes 2700 2100 0    60   ~ 0
+ISP tool (In system programmer)
+Text Notes 4850 7150 0    60   ~ 0
+Reset circuit\nstartup in 0.1[sec]
+Text Notes 1350 1900 0    60   ~ 0
+9V in - 170V out, 5V out
 $EndSCHEMATC

Commit message: 部品リスト・パッケージライブラリを更新
Parts:
- R1: value R -> 510
- R4, R5: value R -> 10k
- renumbered C13 to C2, C2 to C3, C3 to C4, C4 to C5
Changed lines of the file:
@@
 P 2150 3300
 F 0 "R1" V 2230 3300 40  0000 C CNN
-F 1 "R" V 2157 3301 40  0000 C CNN
+F 1 "510" V 2157 3301 40  0000 C CNN
 F 2 "~" V 2080 3300 30  0000 C CNN
 F 3 "~" H 2150 3300 30  0000 C CNN
@@
 $EndComp
 $Comp
-L C C4
+L C C5
 U 1 1 53F8D40A
 P 6300 3900
-F 0 "C4" H 6300 4000 40  0000 L CNN
+F 0 "C5" H 6300 4000 40  0000 L CNN
 F 1 "22p" H 6306 3815 40  0000 L CNN
 F 2 "~" H 6338 3750 30  0000 C CNN
@@
 $EndComp
 $Comp
-L C C3
+L C C4
 U 1 1 53F8D419
 P 5700 3900
-F 0 "C3" H 5700 4000 40  0000 L CNN
+F 0 "C4" H 5700 4000 40  0000 L CNN
 F 1 "22p" H 5706 3815 40  0000 L CNN
 F 2 "~" H 5738 3750 30  0000 C CNN
@@
 $EndComp
 $Comp
-L C C2
+L C C3
 U 1 1 53F90D20
 P 5200 6600
-F 0 "C2" H 5200 6700 40  0000 L CNN
+F 0 "C3" H 5200 6700 40  0000 L CNN
 F 1 "10u" H 5050 6500 40  0000 L CNN
 F 2 "~" H 5238 6450 30  0000 C CNN
@@
 P 6850 1850
 F 0 "R4" V 6930 1850 40  0000 C CNN
-F 1 "R" V 6857 1851 40  0000 C CNN
+F 1 "10k" V 6857 1851 40  0000 C CNN
 F 2 "~" V 6780 1850 30  0000 C CNN
 F 3 "~" H 6850 1850 30  0000 C CNN
@@
 P 7000 1950
 F 0 "R5" V 7080 1950 40  0000 C CNN
-F 1 "R" V 7007 1951 40  0000 C CNN
+F 1 "10k" V 7007 1951 40  0000 C CNN
 F 2 "~" V 6930 1950 30  0000 C CNN
 F 3 "~" H 7000 1950 30  0000 C CNN
@@
 	4750 3400 4850 3300
 $Comp
-L C C13
+L C C2
 U 1 1 53FB7281
 P 2400 3850
-F 0 "C13" H 2400 3950 40  0000 L CNN
+F 0 "C2" H 2400 3950 40  0000 L CNN
 F 1 "0.1u" H 2406 3765 40  0000 L CNN
 F 2 "~" H 2438 3700 30  0000 C CNN

Commit message: 部品リスト完了、PCBに部品を配置
Parts:
- X1: value CRYSTAL -> 12MHz
Changed lines of the file:
@@
 Sheet 1 13
 Title ""
-Date "26 aug 2014"
+Date "28 aug 2014"
 Rev ""
 Comp ""
@@
 P 6000 3700
 F 0 "X1" H 6000 3850 60  0000 C CNN
-F 1 "CRYSTAL" H 6000 3550 60  0000 C CNN
+F 1 "12MHz" H 6000 3550 60  0000 C CNN
 F 2 "~" H 6000 3700 60  0000 C CNN
 F 3 "~" H 6000 3700 60  0000 C CNN

Commit message: PCB更新
Parts:
- added U15, U16, U17, U18: MY_PIN52, symbol MY_PIN52
Other:
- note added: "lower board"
- note added: "upper board"
Changed lines of the file:
@@
 Sheet 1 13
 Title ""
-Date "28 aug 2014"
+Date "30 aug 2014"
 Rev ""
 Comp ""
@@
 Text Notes 1350 1900 0    60   ~ 0
 9V in - 170V out, 5V out
+$Comp
+L MY_PIN52 U17
+U 1 1 540098C7
+P 2950 6150
+F 0 "U17" H 2900 5900 60  0000 C CNN
+F 1 "MY_PIN52" V 2950 6200 60  0000 C CNN
+F 2 "" H 2950 6150 60  0000 C CNN
+F 3 "" H 2950 6150 60  0000 C CNN
+	1    2950 6150
+	1    0    0    -1
+$EndComp
+$Comp
+L MY_PIN52 U15
+U 1 1 540098D6
+P 1800 6150
+F 0 "U15" H 1750 5900 60  0000 C CNN
+F 1 "MY_PIN52" V 1800 6200 60  0000 C CNN
+F 2 "" H 1800 6150 60  0000 C CNN
+F 3 "" H 1800 6150 60  0000 C CNN
+	1    1800 6150
+	1    0    0    -1
+$EndComp
+$Comp
+L MY_PIN52 U18
+U 1 1 54009923
+P 2950 7200
+F 0 "U18" H 2900 6950 60  0000 C CNN
+F 1 "MY_PIN52" V 2950 7250 60  0000 C CNN
+F 2 "" H 2950 7200 60  0000 C CNN
+F 3 "" H 2950 7200 60  0000 C CNN
+	1    2950 7200
+	1    0    0    -1
+$EndComp
+$Comp
+L MY_PIN52 U16
+U 1 1 54009929
+P 1800 7200
+F 0 "U16" H 1750 6950 60  0000 C CNN
+F 1 "MY_PIN52" V 1800 7250 60  0000 C CNN
+F 2 "" H 1800 7200 60  0000 C CNN
+F 3 "" H 1800 7200 60  0000 C CNN
+	1    1800 7200
+	1    0    0    -1
+$EndComp
+Wire Notes Line
+	3400 6450 1200 6450
+Wire Notes Line
+	1200 6450 1200 5700
+Wire Notes Line
+	1200 5700 3400 5700
+Wire Notes Line
+	3400 5700 3400 6450
+Wire Notes Line
+	1200 6800 3400 6800
+Wire Notes Line
+	3400 6800 3400 7500
+Wire Notes Line
+	3400 7500 1200 7500
+Wire Notes Line
+	1200 7500 1200 6800
+Text Notes 1200 5650 0    60   ~ 0
+upper board
+Text Notes 1200 6750 0    60   ~ 0
+lower board
 $EndSCHEMATC

Commit message: PCB
Connections:
- net +5V: now also U15.10
- net GND: now also U15.2, U15.3, U15.4, U15.5, U17.10, U17.6, U17.7, U17.8, U17.9
- net MISO: now also U17.5
- net MOSI: now also U17.4
- net PB0: now also U17.1
- net PB1: now also U17.2
- net PB2: now also U17.3
- net PC0: now also U15.9
- net PC1: now also U15.8
- net PC2: now also U15.7
- net PC3: now also U15.6
- net CLK_PW_H: now reaches U15.1
- net PB_P0: now reaches U18.1
- net GND_L: now reaches U18.10
- net GND_L: now also U16.2, U16.3, U16.4, U16.5, U18.6, U18.7, U18.8, U18.9
- net PB_P1: now reaches U18.2
- net PB_P2: now reaches U18.3
- net PB_P3: now reaches U18.4
- net PB_P4: now reaches U18.5
- net CLK_PW_L: now reaches U16.1
- net 5V_L: now reaches U16.10
- net PC_P3: now reaches U16.6
- net PC_P2: now reaches U16.7
- net PC_P1: now reaches U16.8
- net PC_P0: now reaches U16.9
- net Sheet53F905A8/CLKOUT renamed PD0
- net Sheet53F905A8/SCL renamed SDA
- net Sheet53F905A8/SDA renamed SCL
Other:
- moved on the sheet: C1, C2, C3, C4, C5, D1, IC1, P1, R1, R2, R3, R4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
