File: files/pcb/kicad/kicad_project.sch (KiCad schematic (older format))
At the start: 18 parts, among them IC1 ATMEGA328-A, P1 CONN_6, U15 MY_PIN52, U16 MY_PIN52, U17 MY_PIN52, U18 MY_PIN52, X1 12MHz

Commit message: PCB更新
Connections:
- net +5V: now also U16.6; no longer U16.10
- net +9V: now also U16.4
- net ADC6: now also U16.10; no longer U16.9
- net PD4: now also U16.9; no longer U16.8
- net PIN5V: now also U15.6; no longer U15.10
- net PIN9V: now also U15.4
- net PINADC6: now also U15.10; no longer U15.9
- net PINCLKOUT: now also U15.9; no longer U15.8
- net PINSCL: now also U15.7; no longer U15.6
- net PINSDA: now also U15.8; no longer U15.7
- net SCL: now also U16.7; no longer U16.6
- net SDA: now also U16.8; no longer U16.7
- no-connect marks 15 -> 13
Other:
- moved on the sheet: U15
Changed lines of the file:
@@
 Sheet 1 8
 Title ""
-Date "2 sep 2014"
+Date "4 sep 2014"
 Rev ""
 Comp ""
@@
 L MY_PIN52 U15
 U 1 1 540098D6
-P 7950 4950
-F 0 "U15" H 7900 4700 60  0000 C CNN
-F 1 "MY_PIN52" V 7950 5000 60  0000 C CNN
-F 2 "" H 7950 4950 60  0000 C CNN
-F 3 "" H 7950 4950 60  0000 C CNN
-	1    7950 4950
+P 7700 4950
+F 0 "U15" H 7650 4700 60  0000 C CNN
+F 1 "MY_PIN52" V 7700 5000 60  0000 C CNN
+F 2 "" H 7700 4950 60  0000 C CNN
+F 3 "" H 7700 4950 60  0000 C CNN
+	1    7700 4950
 	1    0    0    -1
 $EndComp
@@
 Text Label 8150 3700 0    60   ~ 0
 SDA
-Text GLabel 8450 4600 2    60   Input ~ 0
+Text GLabel 8200 5200 2    60   Input ~ 0
 PIN5V
 $Comp
 L +5V #PWR011
 U 1 1 54045B6C
-P 8250 6050
-F 0 "#PWR011" H 8250 6140 20  0001 C CNN
-F 1 "+5V" H 8250 6140 30  0000 C CNN
-F 2 "" H 8250 6050 60  0000 C CNN
-F 3 "" H 8250 6050 60  0000 C CNN
-	1    8250 6050
+P 8250 6550
+F 0 "#PWR011" H 8250 6640 20  0001 C CNN
+F 1 "+5V" H 8250 6640 30  0000 C CNN
+F 2 "" H 8250 6550 60  0000 C CNN
+F 3 "" H 8250 6550 60  0000 C CNN
+	1    8250 6550
 	1    0    0    -1
 $EndComp
@@
 	1    0    0    -1
 $EndComp
-Text GLabel 7400 5200 0    60   Input ~ 0
+Text GLabel 7150 5200 0    60   Input ~ 0
 PINGND
 $Comp
@@
 	1    0    0    -1
 $EndComp
+Text Label 8250 6350 0    60   ~ 0
+SDA
 Text Label 8250 6450 0    60   ~ 0
-SDA
-Text Label 8250 6550 0    60   ~ 0
 SCL
 Connection ~ 2600 6050
@@
 Wire Notes Line
 	7550 2500 8600 2500
-Wire Wire Line
-	8300 4700 8400 4700
-Wire Wire Line
-	8250 6050 8250 6150
 Wire Notes Line
 	8950 2500 10000 2500
-Text GLabel 8450 5200 2    60   Input ~ 0
+Text GLabel 8200 5050 2    60   Input ~ 0
 PINSCL
-Text GLabel 8450 5050 2    60   Input ~ 0
+Text GLabel 8200 4900 2    60   Input ~ 0
 PINSDA
 Wire Wire Line
-	8400 5100 8400 5200
-Wire Wire Line
-	8400 5200 8450 5200
+	8150 5100 8150 5200
+Wire Wire Line
+	8150 5200 8200 5200
 Wire Notes Line
 	8950 1000 10150 1000
@@
 Wire Wire Line
 	8000 1600 7750 1600
-Text Label 8250 6350 0    60   ~ 0
+Text Label 8250 6250 0    60   ~ 0
 PD4
-Text GLabel 8450 4900 2    60   Input ~ 0
+Text GLabel 8350 4700 2    60   Input ~ 0
 PINCLKOUT
 Wire Wire Line
-	8450 5050 8400 5050
-Wire Wire Line
-	8400 5050 8400 5000
-Wire Wire Line
-	8400 5000 8300 5000
-Wire Wire Line
-	8300 5100 8400 5100
-Wire Wire Line
-	8450 4900 8300 4900
+	8200 5050 8150 5050
+Wire Wire Line
+	8150 5050 8150 5000
+Wire Wire Line
+	8150 5000 8050 5000
+Wire Wire Line
+	8050 5100 8150 5100
+Wire Wire Line
+	8200 4900 8050 4900
 $Comp
 L +9V #PWR017
@@
 Wire Wire Line
 	7500 6750 7500 6550
-NoConn ~ 7550 5000
 NoConn ~ 9550 4800
 NoConn ~ 9550 4900
@@
 NoConn ~ 9650 6300
 NoConn ~ 9650 6400
-NoConn ~ 7500 6450
-NoConn ~ 4650 5650
-NoConn ~ 4650 5550
 Text Label 2250 5300 0    60   ~ 0
 ADC6
 Wire Wire Line
 	2750 5300 2250 5300
-Text Label 8250 6250 0    60   ~ 0
+Text Label 8250 6150 0    60   ~ 0
 ADC6
-Wire Wire Line
-	8300 4800 8400 4800
-Wire Wire Line
-	8400 4800 8400 4750
-Wire Wire Line
-	8400 4750 8450 4750
-Text GLabel 8450 4750 2    60   Input ~ 0
+Text GLabel 8150 4550 2    60   Input ~ 0
 PINADC6
-Wire Wire Line
-	8400 4700 8400 4600
-Wire Wire Line
-	8400 4600 8450 4600
 Text GLabel 7750 2150 0    60   Input ~ 0
 PINADC6
@@
 PD7
 Wire Wire Line
-	7500 6350 7350 6350
+	7350 6350 7500 6350
 Wire Wire Line
 	7350 6250 7500 6250
 Wire Wire Line
 	7500 6150 7350 6150
-Text GLabel 7400 4600 0    60   Input ~ 0
+Text GLabel 7150 4600 0    60   Input ~ 0
 PINPD5
-Text GLabel 7400 4750 0    60   Input ~ 0
+Text GLabel 7150 4800 0    60   Input ~ 0
 PINPD6
-Text GLabel 7400 4900 0    60   Input ~ 0
+Text GLabel 6700 4900 0    60   Input ~ 0
 PINPD7
 Wire Wire Line
-	7550 5100 7500 5100
-Wire Wire Line
-	7500 5100 7500 5200
-Wire Wire Line
-	7500 5200 7400 5200
-Wire Wire Line
-	7400 4900 7550 4900
-Wire Wire Line
-	7550 4800 7500 4800
-Wire Wire Line
-	7500 4800 7500 4750
-Wire Wire Line
-	7500 4750 7400 4750
-Wire Wire Line
-	7550 4700 7500 4700
-Wire Wire Line
-	7500 4700 7500 4600
-Wire Wire Line
-	7500 4600 7400 4600
+	7300 5100 7250 5100
+Wire Wire Line
+	7250 5100 7250 5200
+Wire Wire Line
+	7250 5200 7150 5200
+Wire Wire Line
+	7300 4700 7250 4700
+Wire Wire Line
+	7250 4700 7250 4600
+Wire Wire Line
+	7250 4600 7150 4600
 Text GLabel 6100 1300 0    60   Input ~ 0
 PINPD5
@@
 Connection ~ 10400 6200
 Connection ~ 10400 6100
+Wire Wire Line
+	8100 4700 8100 4550
+Wire Wire Line
+	8100 4550 8150 4550
+Wire Wire Line
+	8100 4700 8050 4700
+Wire Wire Line
+	8050 4800 8200 4800
+Wire Wire Line
+	8200 4800 8200 4700
+Wire Wire Line
+	8200 4700 8350 4700
+Wire Wire Line
+	7150 4800 7300 4800
+$Comp
+L +9V #PWR018
+U 1 1 5408AC70
+P 7150 6350
+F 0 "#PWR018" H 7150 6320 20  0001 C CNN
+F 1 "+9V" H 7150 6460 30  0000 C CNN
+F 2 "" H 7150 6350 60  0000 C CNN
+F 3 "" H 7150 6350 60  0000 C CNN
+	1    7150 6350
+	1    0    0    -1
+$EndComp
+Wire Wire Line
+	7500 6450 7150 6450
+Wire Wire Line
+	7150 6450 7150 6350
+Text GLabel 7100 5000 0    60   Input ~ 0
+PIN9V
+Wire Wire Line
+	7050 5400 7100 5400
+Wire Wire Line
+	7100 5000 7300 5000
+Wire Wire Line
+	7300 4900 6700 4900
+NoConn ~ 4650 5550
+NoConn ~ 4650 5650
 $EndSCHEMATC

Commit message: 基板が描けた
Parts:
- added U12, U13: MY_PIN72, symbol MY_PIN72
Connections:
- net labels added: INT0_D+, INT1_D-, PIND+, PIND-, PINPB0, PINPB1, PINPB2, PINPB3, PINPB4, PINPB[0..4], PINPC0, PINPC1, PINPC2, PINPC3, PINPC[0..3]
- net labels removed: PB[0..4], PC[0..3], PINADC6, PINCLKOUT, PINPD5, PINPD6, PINPD7, PINSCL, PINSDA
- wire segments 81 -> 84
- no-connect marks 13 -> 3
Other:
- note added: "USB"
- moved on the sheet: C1, C2, C4, C5, D1, IC1, R1, U15, U16, X1

Commit message: DRC完了
あとはシルク移動かなぁ
Connections:
- wire segments 84 -> 82
Changed lines of the file:
@@
 Sheet 1 8
 Title ""
-Date "5 sep 2014"
+Date "6 sep 2014"
 Rev ""
 Comp ""
@@
 	9600 6500 9650 6500
 Wire Wire Line
-	5900 6800 5900 6600
+	5900 6300 5900 6800
 Wire Wire Line
 	1850 5500 1350 5500
@@
 Connection ~ 5900 6750
 Wire Wire Line
-	5900 6300 5900 6400
-Wire Wire Line
 	5800 6400 5800 6700
 Wire Wire Line
 	5800 6700 5900 6700
 Connection ~ 5900 6700
-Wire Wire Line
-	5800 6400 10400 6400
 Wire Wire Line
 	8450 6300 8950 6300
@@
 Connection ~ 9650 6100
 Connection ~ 9650 6300
+Connection ~ 5900 6600
 $EndSCHEMATC
