File: files/pcb/kicad/napion.sch (KiCad schematic (older format))
At the start: 0 parts

Commit message: 回路図ERC途中
Parts:
- added U13: SENSOR, ~, symbol SENSOR
Connections:
- new net +5V: U13.1 (VCC)
- new net GND: U13.2 (GND)
- new net out: U13.3 (OUT)
Changed lines of the file:
@@
 $Descr A4 11693 8268
 encoding utf-8
-Sheet 1 13
+Sheet 10 13
 Title ""
-Date "24 aug 2014"
+Date "25 aug 2014"
 Rev ""
 Comp ""
@@
 Comment4 ""
 $EndDescr
+$Comp
+L SENSOR U13
+U 1 1 53FB5E8C
+P 5850 3750
+F 0 "U13" H 5950 3500 39  0000 C CNN
+F 1 "SENSOR" H 5700 3500 39  0000 C CNN
+F 2 "~" H 5550 3600 60  0000 C CNN
+F 3 "~" H 5550 3600 60  0000 C CNN
+	1    5850 3750
+	-1   0    0    -1
+$EndComp
+$Comp
+L GND #PWR049
+U 1 1 53FB5E9B
+P 5850 4300
+F 0 "#PWR049" H 5850 4300 30  0001 C CNN
+F 1 "GND" H 5850 4230 30  0001 C CNN
+F 2 "" H 5850 4300 60  0000 C CNN
+F 3 "" H 5850 4300 60  0000 C CNN
+	1    5850 4300
+	1    0    0    -1
+$EndComp
+$Comp
+L +5V #PWR050
+U 1 1 53FB5EB9
+P 5850 3200
+F 0 "#PWR050" H 5850 3290 20  0001 C CNN
+F 1 "+5V" H 5850 3290 30  0000 C CNN
+F 2 "" H 5850 3200 60  0000 C CNN
+F 3 "" H 5850 3200 60  0000 C CNN
+	1    5850 3200
+	1    0    0    -1
+$EndComp
+Text HLabel 5300 3750 0    60   Input ~ 0
+out
+Wire Wire Line
+	5850 4250 5850 4300
+Wire Wire Line
+	5850 3250 5850 3200
+Wire Wire Line
+	5400 3750 5300 3750
 $EndSCHEMATC

Commit message: 部品リスト・パッケージライブラリを更新
Parts:
- renumbered U13 to U14
Changed lines of the file:
@@
 $EndDescr
 $Comp
-L SENSOR U13
+L SENSOR U14
 U 1 1 53FB5E8C
 P 5850 3750
-F 0 "U13" H 5950 3500 39  0000 C CNN
+F 0 "U14" H 5950 3500 39  0000 C CNN
 F 1 "SENSOR" H 5700 3500 39  0000 C CNN
 F 2 "~" H 5550 3600 60  0000 C CNN
@@
 $EndComp
 $Comp
-L GND #PWR057
+L GND #PWR060
 U 1 1 53FB5E9B
 P 5850 4300
-F 0 "#PWR057" H 5850 4300 30  0001 C CNN
+F 0 "#PWR060" H 5850 4300 30  0001 C CNN
 F 1 "GND" H 5850 4230 30  0001 C CNN
 F 2 "" H 5850 4300 60  0000 C CNN
@@
 $EndComp
 $Comp
-L +5V #PWR058
+L +5V #PWR061
 U 1 1 53FB5EB9
 P 5850 3200
-F 0 "#PWR058" H 5850 3290 20  0001 C CNN
+F 0 "#PWR061" H 5850 3290 20  0001 C CNN
 F 1 "+5V" H 5850 3290 30  0000 C CNN
 F 2 "" H 5850 3200 60  0000 C CNN

Commit message: 部品リスト完了、PCBに部品を配置
Parts:
- added C17: 0.1u, ~, symbol C
- U14: value SENSOR -> napion
Connections:
- net +5V: now also C17.1
- net GND: now also C17.2
Changed lines of the file:
@@
 Sheet 10 13
 Title ""
-Date "26 aug 2014"
+Date "28 aug 2014"
 Rev ""
 Comp ""
@@
 P 5850 3750
 F 0 "U14" H 5950 3500 39  0000 C CNN
-F 1 "SENSOR" H 5700 3500 39  0000 C CNN
+F 1 "napion" H 5700 3500 39  0000 C CNN
 F 2 "~" H 5550 3600 60  0000 C CNN
 F 3 "~" H 5550 3600 60  0000 C CNN
@@
 Wire Wire Line
 	5400 3750 5300 3750
+$Comp
+L C C17
+U 1 1 53FF6211
+P 6250 3750
+F 0 "C17" H 6250 3850 40  0000 L CNN
+F 1 "0.1u" H 6256 3665 40  0000 L CNN
+F 2 "~" H 6288 3600 30  0000 C CNN
+F 3 "~" H 6250 3750 60  0000 C CNN
+	1    6250 3750
+	1    0    0    -1
+$EndComp
+Wire Wire Line
+	5850 3250 6250 3250
+Wire Wire Line
+	6250 3250 6250 3550
+Wire Wire Line
+	6250 3950 6250 4250
+Wire Wire Line
+	6250 4250 5850 4250
 $EndSCHEMATC
