File: files/pcb/kicad/switch.sch (KiCad schematic (older format))
At the start: 0 parts

Commit message: 回路図更新
温度湿度センサ
大気圧センサ
輝度センサ
Parts:
- added R? (x3): 10k, ~, symbol R
- added SW?: EVQWK, symbol EVQWK
Connections:
- new net +5V: R?.1, R?.1, R?.1
- new net A: R?.2, SW?.1 (A)
- new net B: R?.2, SW?.6 (B)
- new net GND: SW?.2 (com), SW?.3 (SW1), SW?.5 (SW1)
- new net Push: R?.2, SW?.4 (SW2)
Changed lines of the file:
@@
 $Descr A4 11693 8268
 encoding utf-8
-Sheet 1 12
+Sheet 6 12
 Title ""
 Date "23 aug 2014"
@@
 Comment4 ""
 $EndDescr
+Text HLabel 5000 4000 0    60   Input ~ 0
+A
+Text HLabel 5000 4500 0    60   Input ~ 0
+B
+Text HLabel 5000 4300 0    60   Input ~ 0
+Push
+Wire Wire Line
+	5000 4000 6100 4000
+Wire Wire Line
+	5000 4500 6100 4500
+Wire Wire Line
+	5000 4300 6100 4300
+$Comp
+L R R?
+U 1 1 53F91538
+P 5550 3650
+F 0 "R?" V 5630 3650 40  0000 C CNN
+F 1 "10k" V 5557 3651 40  0000 C CNN
+F 2 "~" V 5480 3650 30  0000 C CNN
+F 3 "~" H 5550 3650 30  0000 C CNN
+	1    5550 3650
+	1    0    0    -1
+$EndComp
+$Comp
+L R R?
+U 1 1 53F91546
+P 5350 3650
+F 0 "R?" V 5430 3650 40  0000 C CNN
+F 1 "10k" V 5357 3651 40  0000 C CNN
+F 2 "~" V 5280 3650 30  0000 C CNN
+F 3 "~" H 5350 3650 30  0000 C CNN
+	1    5350 3650
+	1    0    0    -1
+$EndComp
+$Comp
+L R R?
+U 1 1 53F9154E
+P 5150 3650
+F 0 "R?" V 5230 3650 40  0000 C CNN
+F 1 "10k" V 5157 3651 40  0000 C CNN
+F 2 "~" V 5080 3650 30  0000 C CNN
+F 3 "~" H 5150 3650 30  0000 C CNN
+	1    5150 3650
+	1    0    0    -1
+$EndComp
+Wire Wire Line
+	5550 3900 5550 4300
+Connection ~ 5550 4300
+Wire Wire Line
+	5350 3900 5350 4500
+Connection ~ 5350 4500
+Wire Wire Line
+	5150 3900 5150 4000
+Connection ~ 5150 4000
+$Comp
+L +5V #PWR?
+U 1 1 53F9157F
+P 5150 3250
+F 0 "#PWR?" H 5150 3340 20  0001 C CNN
+F 1 "+5V" H 5150 3340 30  0000 C CNN
+F 2 "" H 5150 3250 60  0000 C CNN
+F 3 "" H 5150 3250 60  0000 C CNN
+	1    5150 3250
+	1    0    0    -1
+$EndComp
+Wire Wire Line
+	5150 3250 5150 3400
+Wire Wire Line
+	5350 3400 5350 3300
+Wire Wire Line
+	5150 3300 5550 3300
+Connection ~ 5150 3300
+Wire Wire Line
+	5550 3300 5550 3400
+Connection ~ 5350 3300
+$Comp
+L EVQWK SW?
+U 1 1 53F918EF
+P 6500 4250
+F 0 "SW?" H 6600 4650 39  0000 C CNN
+F 1 "EVQWK" H 6600 3900 39  0000 C CNN
+F 2 "" H 6500 4250 60  0000 C CNN
+F 3 "" H 6500 4250 60  0000 C CNN
+	1    6500 4250
+	1    0    0    -1
+$EndComp
+$Comp
+L GND #PWR?
+U 1 1 53F91903
+P 5950 4700
+F 0 "#PWR?" H 5950 4700 30  0001 C CNN
+F 1 "GND" H 5950 4630 30  0001 C CNN
+F 2 "" H 5950 4700 60  0000 C CNN
+F 3 "" H 5950 4700 60  0000 C CNN
+	1    5950 4700
+	1    0    0    -1
+$EndComp
+Wire Wire Line
+	5950 4100 5950 4700
+Wire Wire Line
+	5950 4400 6100 4400
+Wire Wire Line
+	5950 4200 6100 4200
+Connection ~ 5950 4400
+Wire Wire Line
+	5950 4100 6100 4100
+Connection ~ 5950 4200
 $EndSCHEMATC

Commit message: 回路図更新、DS1307対応
バスの接続が未
Parts:
- gave numbers to parts that had none: 4
Changed lines of the file:
@@
 $Descr A4 11693 8268
 encoding utf-8
-Sheet 6 12
+Sheet 6 13
 Title ""
-Date "23 aug 2014"
+Date "24 aug 2014"
 Rev ""
 Comp ""
@@
 	5000 4300 6100 4300
 $Comp
-L R R?
+L R R22
 U 1 1 53F91538
 P 5550 3650
-F 0 "R?" V 5630 3650 40  0000 C CNN
+F 0 "R22" V 5630 3650 40  0000 C CNN
 F 1 "10k" V 5557 3651 40  0000 C CNN
 F 2 "~" V 5480 3650 30  0000 C CNN
@@
 $EndComp
 $Comp
-L R R?
+L R R21
 U 1 1 53F91546
 P 5350 3650
-F 0 "R?" V 5430 3650 40  0000 C CNN
+F 0 "R21" V 5430 3650 40  0000 C CNN
 F 1 "10k" V 5357 3651 40  0000 C CNN
 F 2 "~" V 5280 3650 30  0000 C CNN
@@
 $EndComp
 $Comp
-L R R?
+L R R20
 U 1 1 53F9154E
 P 5150 3650
-F 0 "R?" V 5230 3650 40  0000 C CNN
+F 0 "R20" V 5230 3650 40  0000 C CNN
 F 1 "10k" V 5157 3651 40  0000 C CNN
 F 2 "~" V 5080 3650 30  0000 C CNN
@@
 Connection ~ 5150 4000
 $Comp
-L +5V #PWR?
+L +5V #PWR44
 U 1 1 53F9157F
 P 5150 3250
-F 0 "#PWR?" H 5150 3340 20  0001 C CNN
+F 0 "#PWR44" H 5150 3340 20  0001 C CNN
 F 1 "+5V" H 5150 3340 30  0000 C CNN
 F 2 "" H 5150 3250 60  0000 C CNN
@@
 Connection ~ 5350 3300
 $Comp
-L EVQWK SW?
+L EVQWK SW2
 U 1 1 53F918EF
 P 6500 4250
-F 0 "SW?" H 6600 4650 39  0000 C CNN
+F 0 "SW2" H 6600 4650 39  0000 C CNN
 F 1 "EVQWK" H 6600 3900 39  0000 C CNN
 F 2 "" H 6500 4250 60  0000 C CNN
@@
 $EndComp
 $Comp
-L GND #PWR?
+L GND #PWR45
 U 1 1 53F91903
 P 5950 4700
-F 0 "#PWR?" H 5950 4700 30  0001 C CNN
+F 0 "#PWR45" H 5950 4700 30  0001 C CNN
 F 1 "GND" H 5950 4630 30  0001 C CNN
 F 2 "" H 5950 4700 60  0000 C CNN

Commit message: 部品リスト・パッケージライブラリを更新
Parts:
- added SW3, SW4, SW5: SW_PUSH, ~, symbol SW_PUSH
- renumbered R20 to R24, R21 to R25, R22 to R26
Connections:
- net A: now also SW3.1
- net B: now also SW4.1
- net GND: now also SW3.2, SW4.2, SW5.2
- net Push: now also SW5.1
Other:
- note added: "Push switch or ECQWK"
- moved on the sheet: R24, R26
Changed lines of the file:
@@
 Comment4 ""
 $EndDescr
-Text HLabel 5000 4000 0    60   Input ~ 0
+Text HLabel 4900 4000 0    60   Input ~ 0
 A
-Text HLabel 5000 4500 0    60   Input ~ 0
+Text HLabel 4900 4500 0    60   Input ~ 0
 B
-Text HLabel 5000 4300 0    60   Input ~ 0
+Text HLabel 4900 4300 0    60   Input ~ 0
 Push
 Wire Wire Line
-	5000 4000 6100 4000
+	4900 4000 6100 4000
 Wire Wire Line
-	5000 4500 6100 4500
+	4900 4500 6100 4500
 Wire Wire Line
-	5000 4300 6100 4300
+	4900 4300 6100 4300
 $Comp
-L R R22
+L R R26
 U 1 1 53F91538
-P 5550 3650
-F 0 "R22" V 5630 3650 40  0000 C CNN
-F 1 "10k" V 5557 3651 40  0000 C CNN
-F 2 "~" V 5480 3650 30  0000 C CNN
-F 3 "~" H 5550 3650 30  0000 C CNN
-	1    5550 3650
+P 5650 3650
+F 0 "R26" V 5730 3650 40  0000 C CNN
+F 1 "10k" V 5657 3651 40  0000 C CNN
+F 2 "~" V 5580 3650 30  0000 C CNN
+F 3 "~" H 5650 3650 30  0000 C CNN
+	1    5650 3650
 	1    0    0    -1
 $EndComp
 $Comp
-L R R21
+L R R25
 U 1 1 53F91546
 P 5350 3650
-F 0 "R21" V 5430 3650 40  0000 C CNN
+F 0 "R25" V 5430 3650 40  0000 C CNN
 F 1 "10k" V 5357 3651 40  0000 C CNN
 F 2 "~" V 5280 3650 30  0000 C CNN
@@
 $EndComp
 $Comp
-L R R20
+L R R24
 U 1 1 53F9154E
-P 5150 3650
-F 0 "R20" V 5230 3650 40  0000 C CNN
-F 1 "10k" V 5157 3651 40  0000 C CNN
-F 2 "~" V 5080 3650 30  0000 C CNN
-F 3 "~" H 5150 3650 30  0000 C CNN
-	1    5150 3650
+P 5050 3650
+F 0 "R24" V 5130 3650 40  0000 C CNN
+F 1 "10k" V 5057 3651 40  0000 C CNN
+F 2 "~" V 4980 3650 30  0000 C CNN
+F 3 "~" H 5050 3650 30  0000 C CNN
+	1    5050 3650
 	1    0    0    -1
 $EndComp
 Wire Wire Line
-	5550 3900 5550 4300
-Connection ~ 5550 4300
+	5650 3900 5650 4750
+Connection ~ 5650 4300
 Wire Wire Line
-	5350 3900 5350 4500
+	5350 3900 5350 4750
 Connection ~ 5350 4500
 Wire Wire Line
-	5150 3900 5150 4000
-Connection ~ 5150 4000
+	5050 3900 5050 4750
+Connection ~ 5050 4000
 $Comp
 L +5V #PWR052
 U 1 1 53F9157F
-P 5150 3250
-F 0 "#PWR052" H 5150 3340 20  0001 C CNN
-F 1 "+5V" H 5150 3340 30  0000 C CNN
-F 2 "" H 5150 3250 60  0000 C CNN
-F 3 "" H 5150 3250 60  0000 C CNN
-	1    5150 3250
+P 5050 3250
+F 0 "#PWR052" H 5050 3340 20  0001 C CNN
+F 1 "+5V" H 5050 3340 30  0000 C CNN
+F 2 "" H 5050 3250 60  0000 C CNN
+F 3 "" H 5050 3250 60  0000 C CNN
+	1    5050 3250
 	1    0    0    -1
 $EndComp
 Wire Wire Line
-	5150 3250 5150 3400
+	5050 3250 5050 3400
 Wire Wire Line
 	5350 3400 5350 3300
 Wire Wire Line
-	5150 3300 5550 3300
-Connection ~ 5150 3300
+	5050 3300 5650 3300
+Connection ~ 5050 3300
 Wire Wire Line
-	5550 3300 5550 3400
+	5650 3300 5650 3400
 Connection ~ 5350 3300
 $Comp
@@
 	5950 4100 6100 4100
 Connection ~ 5950 4200
+$Comp
+L SW_PUSH SW3
+U 1 1 53FCBA5A
+P 5050 5050
+F 0 "SW3" H 5200 5160 50  0000 C CNN
+F 1 "SW_PUSH" H 5050 4970 50  0000 C CNN
+F 2 "~" H 5050 5050 60  0000 C CNN
+F 3 "~" H 5050 5050 60  0000 C CNN
+	1    5050 5050
+	0    1    1    0
+$EndComp
+$Comp
+L SW_PUSH SW4
+U 1 1 53FCBA67
+P 5350 5050
+F 0 "SW4" H 5500 5160 50  0000 C CNN
+F 1 "SW_PUSH" H 5350 4970 50  0000 C CNN
+F 2 "~" H 5350 5050 60  0000 C CNN
+F 3 "~" H 5350 5050 60  0000 C CNN
+	1    5350 5050
+	0    1    1    0
+$EndComp
+$Comp
+L SW_PUSH SW5
+U 1 1 53FCBA6D
+P 5650 5050
+F 0 "SW5" H 5800 5160 50  0000 C CNN
+F 1 "SW_PUSH" H 5650 4970 50  0000 C CNN
+F 2 "~" H 5650 5050 60  0000 C CNN
+F 3 "~" H 5650 5050 60  0000 C CNN
+	1    5650 5050
+	0    1    1    0
+$EndComp
+$Comp
+L GND #PWR054
+U 1 1 53FCBB00
+P 5650 5400
+F 0 "#PWR054" H 5650 5400 30  0001 C CNN
+F 1 "GND" H 5650 5330 30  0001 C CNN
+F 2 "" H 5650 5400 60  0000 C CNN
+F 3 "" H 5650 5400 60  0000 C CNN
+	1    5650 5400
+	1    0    0    -1
+$EndComp
+$Comp
+L GND #PWR055
+U 1 1 53FCBB0F
+P 5350 5400
+F 0 "#PWR055" H 5350 5400 30  0001 C CNN
+F 1 "GND" H 5350 5330 30  0001 C CNN
+F 2 "" H 5350 5400 60  0000 C CNN
+F 3 "" H 5350 5400 60  0000 C CNN
+	1    5350 5400
+	1    0    0    -1
+$EndComp
+$Comp
+L GND #PWR056
+U 1 1 53FCBB1E
+P 5050 5400
+F 0 "#PWR056" H 5050 5400 30  0001 C CNN
+F 1 "GND" H 5050 5330 30  0001 C CNN
+F 2 "" H 5050 5400 60  0000 C CNN
+F 3 "" H 5050 5400 60  0000 C CNN
+	1    5050 5400
+	1    0    0    -1
+$EndComp
+Wire Wire Line
+	5650 5350 5650 5400
+Wire Wire Line
+	5350 5350 5350 5400
+Wire Wire Line
+	5050 5350 5050 5400
+Text Notes 6250 5050 0    60   ~ 0
+Push switch or ECQWK
 $EndSCHEMATC
