File: files/pcb/kicad/switch.sch (KiCad schematic (older format))
At the start: 7 parts, among them SW2 EVQWK, SW3 SW_PUSH, SW4 SW_PUSH, SW5 SW_PUSH

Commit message: 必要性の低い部品を削除
機能てんこ盛りよりシンプル小型化のほうがいいかなと思ったので一気に部品を削除
Parts:
- removed SW2: EVQWK, symbol EVQWK
Connections:
- wire segments 17 -> 13
Changed lines of the file:
@@
 $Descr A4 11693 8268
 encoding utf-8
-Sheet 7 13
+Sheet 7 11
 Title ""
 Date "31 aug 2014"
@@
 Connection ~ 5050 4000
 $Comp
-L +5V #PWR037
+L +5V #PWR036
 U 1 1 53F9157F
 P 5050 3250
-F 0 "#PWR037" H 5050 3340 20  0001 C CNN
+F 0 "#PWR036" H 5050 3340 20  0001 C CNN
 F 1 "+5V" H 5050 3340 30  0000 C CNN
 F 2 "" H 5050 3250 60  0000 C CNN
@@
 	5650 3300 5650 3400
 Connection ~ 5350 3300
-$Comp
-L EVQWK SW2
-U 1 1 53F918EF
-P 6500 4250
-F 0 "SW2" H 6600 4650 39  0000 C CNN
-F 1 "EVQWK" H 6600 3900 39  0000 C CNN
-F 2 "" H 6500 4250 60  0000 C CNN
-F 3 "" H 6500 4250 60  0000 C CNN
-	1    6500 4250
-	1    0    0    -1
-$EndComp
-$Comp
-L GND #PWR038
-U 1 1 53F91903
-P 5950 4700
-F 0 "#PWR038" H 5950 4700 30  0001 C CNN
-F 1 "GND" H 5950 4630 30  0001 C CNN
-F 2 "" H 5950 4700 60  0000 C CNN
-F 3 "" H 5950 4700 60  0000 C CNN
-	1    5950 4700
-	1    0    0    -1
-$EndComp
-Wire Wire Line
-	5950 4100 5950 4700
-Wire Wire Line
-	5950 4400 6100 4400
-Wire Wire Line
-	5950 4200 6100 4200
-Connection ~ 5950 4400
-Wire Wire Line
-	5950 4100 6100 4100
-Connection ~ 5950 4200
 $Comp
 L SW_PUSH SW3
@@
 $EndComp
 $Comp
-L GND #PWR039
+L GND #PWR037
 U 1 1 53FCBB00
 P 5650 5400
-F 0 "#PWR039" H 5650 5400 30  0001 C CNN
+F 0 "#PWR037" H 5650 5400 30  0001 C CNN
 F 1 "GND" H 5650 5330 30  0001 C CNN
 F 2 "" H 5650 5400 60  0000 C CNN
@@
 $EndComp
 $Comp
-L GND #PWR040
+L GND #PWR038
 U 1 1 53FCBB0F
 P 5350 5400
-F 0 "#PWR040" H 5350 5400 30  0001 C CNN
+F 0 "#PWR038" H 5350 5400 30  0001 C CNN
 F 1 "GND" H 5350 5330 30  0001 C CNN
 F 2 "" H 5350 5400 60  0000 C CNN
@@
 $EndComp
 $Comp
-L GND #PWR041
+L GND #PWR039
 U 1 1 53FCBB1E
 P 5050 5400
-F 0 "#PWR041" H 5050 5400 30  0001 C CNN
+F 0 "#PWR039" H 5050 5400 30  0001 C CNN
 F 1 "GND" H 5050 5330 30  0001 C CNN
 F 2 "" H 5050 5400 60  0000 C CNN

Commit message: 設計見直し
部品見直し
USB・DCジャック自動切り替え
マイコンを下段のボードに移動
ニキシー管駆動電源を上段ボードに移動
Connections:
- net labels added: PIN5V, PINGND
- net labels removed: +5V, GND
- wire segments 13 -> 14
Changed lines of the file:
@@
 $Descr A4 11693 8268
 encoding utf-8
-Sheet 7 11
+Sheet 7 8
 Title ""
-Date "31 aug 2014"
+Date "1 sep 2014"
 Rev ""
 Comp ""
@@
 	5050 3900 5050 4750
 Connection ~ 5050 4000
-$Comp
-L +5V #PWR036
-U 1 1 53F9157F
-P 5050 3250
-F 0 "#PWR036" H 5050 3340 20  0001 C CNN
-F 1 "+5V" H 5050 3340 30  0000 C CNN
-F 2 "" H 5050 3250 60  0000 C CNN
-F 3 "" H 5050 3250 60  0000 C CNN
-	1    5050 3250
-	1    0    0    -1
-$EndComp
-Wire Wire Line
-	5050 3250 5050 3400
 Wire Wire Line
 	5350 3400 5350 3300
 Wire Wire Line
-	5050 3300 5650 3300
+	4750 3300 5650 3300
 Connection ~ 5050 3300
 Wire Wire Line
@@
 	0    1    1    0
 $EndComp
-$Comp
-L GND #PWR037
-U 1 1 53FCBB00
-P 5650 5400
-F 0 "#PWR037" H 5650 5400 30  0001 C CNN
-F 1 "GND" H 5650 5330 30  0001 C CNN
-F 2 "" H 5650 5400 60  0000 C CNN
-F 3 "" H 5650 5400 60  0000 C CNN
-	1    5650 5400
-	1    0    0    -1
-$EndComp
-$Comp
-L GND #PWR038
-U 1 1 53FCBB0F
-P 5350 5400
-F 0 "#PWR038" H 5350 5400 30  0001 C CNN
-F 1 "GND" H 5350 5330 30  0001 C CNN
-F 2 "" H 5350 5400 60  0000 C CNN
-F 3 "" H 5350 5400 60  0000 C CNN
-	1    5350 5400
-	1    0    0    -1
-$EndComp
-$Comp
-L GND #PWR039
-U 1 1 53FCBB1E
-P 5050 5400
-F 0 "#PWR039" H 5050 5400 30  0001 C CNN
-F 1 "GND" H 5050 5330 30  0001 C CNN
-F 2 "" H 5050 5400 60  0000 C CNN
-F 3 "" H 5050 5400 60  0000 C CNN
-	1    5050 5400
-	1    0    0    -1
-$EndComp
 Wire Wire Line
-	5650 5350 5650 5400
+	5650 5450 5650 5350
 Wire Wire Line
-	5350 5350 5350 5400
+	5350 5450 5350 5350
 Wire Wire Line
-	5050 5350 5050 5400
-Text Notes 6250 5050 0    60   ~ 0
+	5050 5350 5050 5450
+Text Notes 6250 4350 0    60   ~ 0
 Push switch or ECQWK
+Text GLabel 4750 3300 0    60   Input ~ 0
+PIN5V
+Text GLabel 4750 5450 0    60   Input ~ 0
+PINGND
+Wire Wire Line
+	4750 5450 5650 5450
+Connection ~ 5350 5450
+Connection ~ 5050 5450
+Wire Wire Line
+	5050 3400 5050 3300
 $EndSCHEMATC
