File: files/pcb/kicad/nixie.sch (KiCad schematic (older format))
At the start: 1 part

Commit message: 回路図更新、DS1307対応
バスの接続が未
Parts:
- removed VR3: VOLUME, ~, symbol VOLUME
- added IC10, IC9: IC_4PIN, ~, symbol IC_4PIN
- added IC11: SN74141_K155NA, ~, symbol IC_16PIN
- added IC7, IC8: TLP627-4, ~, symbol IC_16PIN
- added R25: 330, ~, symbol R
- added R26, R6: 10k, ~, symbol R
- added R27, R28: 500k, ~, symbol R
- added U2: 74LS138, ~, symbol 74LS138
- added V2: 170V, ~, symbol 170V
Connections:
- net labels added: +5V, GND, cathode_bus, driver_bus
- net labels removed: 170V
- wire segments 4 -> 112
Other:
- note added: "1: 8\n2: 9\n3: A \n4: D\n5: VCC\n6: B\n7: C\n8: 2\n9: 3\n10: 7\n11: 6\n12: GND\n13: 4\n14: 5\n15: 1\n16: 0"

Commit message: 回路図ERC途中
Parts:
- removed U2: 74LS138, ~, symbol 74LS138
- removed V2: 170V, ~, symbol 170V
- added C14: C, ~, symbol C
- added IC13: IC_16PIN, ~, symbol IC_16PIN
Connections:
- net labels added: 170V, N0, N1, N2, N3, N4, N5, N6, N7, N8, N9, N[0..9], PB0, PB1, PB2, PB3, PB4, PB[0..4], PC0, PC1, PC2, PC3, PC[0..3]
- net labels removed: cathode_bus, driver_bus
- wire segments 112 -> 118
Other:
- moved on the sheet: IC10, IC11, IC7, IC8, IC9, R25, R26, R27, R28, R6

Commit message: 部品リスト・パッケージライブラリを更新
Parts:
- added C15: 0.1u, ~, symbol C
- C6: renamed from C14; value C -> 0.1u
- renumbered IC13 to IC2, IC9 to IC3, IC10 to IC4, IC11 to IC5, IC7 to IC6, IC8 to IC7, R28 to R10, R25 to R6, R6 to R7, R26 to R8, R27 to R9
Connections:
- net +5V: now also C6.2, C15.1; no longer C6.1, IC2.6
- net GND: now also C6.1, IC2.6, C15.2; no longer C6.2
Other:
- moved on the sheet: C6
Changed lines of the file:
@@
 PB[0..4]
 $Comp
-L IC_16PIN IC11
+L IC_16PIN IC5
 U 1 1 53F99A7D
 P 4800 6250
-F 0 "IC11" H 4800 6700 39  0000 C CNN
+F 0 "IC5" H 4800 6700 39  0000 C CNN
 F 1 "SN74141_K155NA" V 4800 6250 39  0000 C CNN
 F 2 "~" H 5000 5850 60  0000 C CNN
@@
 L +5V #PWR015
 U 1 1 53F99ADE
-P 4250 5700
-F 0 "#PWR015" H 4250 5790 20  0001 C CNN
-F 1 "+5V" H 4250 5790 30  0000 C CNN
-F 2 "" H 4250 5700 60  0000 C CNN
-F 3 "" H 4250 5700 60  0000 C CNN
-	1    4250 5700
+P 4250 5600
+F 0 "#PWR015" H 4250 5690 20  0001 C CNN
+F 1 "+5V" H 4250 5690 30  0000 C CNN
+F 2 "" H 4250 5600 60  0000 C CNN
+F 3 "" H 4250 5600 60  0000 C CNN
+	1    4250 5600
 	1    0    0    -1
 $EndComp
@@
 L GND #PWR017
 U 1 1 53F99C2C
-P 2700 3150
-F 0 "#PWR017" H 2700 3150 30  0001 C CNN
-F 1 "GND" H 2700 3080 30  0001 C CNN
-F 2 "" H 2700 3150 60  0000 C CNN
-F 3 "" H 2700 3150 60  0000 C CNN
-	1    2700 3150
+P 2700 2800
+F 0 "#PWR017" H 2700 2800 30  0001 C CNN
+F 1 "GND" H 2700 2730 30  0001 C CNN
+F 2 "" H 2700 2800 60  0000 C CNN
+F 3 "" H 2700 2800 60  0000 C CNN
+	1    2700 2800
 	1    0    0    -1
 $EndComp
@@
 L +5V #PWR018
 U 1 1 53F99C3B
-P 2850 1600
-F 0 "#PWR018" H 2850 1690 20  0001 C CNN
-F 1 "+5V" H 2850 1690 30  0000 C CNN
-F 2 "" H 2850 1600 60  0000 C CNN
-F 3 "" H 2850 1600 60  0000 C CNN
-	1    2850 1600
+P 4000 1450
+F 0 "#PWR018" H 4000 1540 20  0001 C CNN
+F 1 "+5V" H 4000 1540 30  0000 C CNN
+F 2 "" H 4000 1450 60  0000 C CNN
+F 3 "" H 4000 1450 60  0000 C CNN
+	1    4000 1450
 	1    0    0    -1
 $EndComp
@@
 $EndComp
 $Comp
-L R R6
+L R R7
 U 1 1 53F99D05
 P 4550 1150
-F 0 "R6" V 4630 1150 40  0000 C CNN
+F 0 "R7" V 4630 1150 40  0000 C CNN
 F 1 "10k" V 4557 1151 40  0000 C CNN
 F 2 "~" V 4480 1150 30  0000 C CNN
@@
 $EndComp
 $Comp
-L IC_16PIN IC8
+L IC_16PIN IC7
 U 1 1 53F9A144
 P 5100 2750
-F 0 "IC8" H 5100 3200 39  0000 C CNN
+F 0 "IC7" H 5100 3200 39  0000 C CNN
 F 1 "TLP627-4" V 5100 2750 39  0000 C CNN
 F 2 "~" H 5300 2350 60  0000 C CNN
@@
 $EndComp
 $Comp
-L R R26
+L R R8
 U 1 1 53F9DAA3
 P 5650 1150
-F 0 "R26" V 5730 1150 40  0000 C CNN
+F 0 "R8" V 5730 1150 40  0000 C CNN
 F 1 "10k" V 5657 1151 40  0000 C CNN
 F 2 "~" V 5580 1150 30  0000 C CNN
@@
 $EndComp
 $Comp
-L IC_16PIN IC7
+L IC_16PIN IC6
 U 1 1 53F9A135
 P 5100 1850
-F 0 "IC7" H 5100 2300 39  0000 C CNN
+F 0 "IC6" H 5100 2300 39  0000 C CNN
 F 1 "TLP627-4" V 5100 1850 39  0000 C CNN
 F 2 "~" H 5300 1450 60  0000 C CNN
@@
 $EndComp
 $Comp
-L R R27
+L R R9
 U 1 1 53FA354D
 P 5650 4900
-F 0 "R27" V 5730 4900 40  0000 C CNN
+F 0 "R9" V 5730 4900 40  0000 C CNN
 F 1 "500k" V 5657 4901 40  0000 C CNN
 F 2 "~" V 5580 4900 30  0000 C CNN
@@
 $EndComp
 $Comp
-L R R28
+L R R10
 U 1 1 53FA3610
 P 5800 4900
-F 0 "R28" V 5880 4900 40  0000 C CNN
+F 0 "R10" V 5880 4900 40  0000 C CNN
 F 1 "500k" V 5807 4901 40  0000 C CNN
 F 2 "~" V 5730 4900 30  0000 C CNN
@@
 $EndComp
 $Comp
-L IC_4PIN IC10
+L IC_4PIN IC4
 U 1 1 53FAC035
 P 4800 4500
-F 0 "IC10" H 4800 4650 39  0000 C CNN
+F 0 "IC4" H 4800 4650 39  0000 C CNN
 F 1 "IC_4PIN" H 4800 4500 39  0000 C CNN
 F 2 "~" H 4750 4350 60  0000 C CNN
@@
 $EndComp
 $Comp
-L IC_4PIN IC9
+L IC_4PIN IC3
 U 1 1 53FAC03B
 P 4800 4150
-F 0 "IC9" H 4800 4300 39  0000 C CNN
+F 0 "IC3" H 4800 4300 39  0000 C CNN
 F 1 "IC_4PIN" H 4800 4150 39  0000 C CNN
 F 2 "~" H 4750 4000 60  0000 C CNN
@@
 $EndComp
 $Comp
-L R R25
+L R R6
 U 1 1 53FAC047
 P 4250 3700
-F 0 "R25" V 4330 3700 40  0000 C CNN
+F 0 "R6" V 4330 3700 40  0000 C CNN
 F 1 "330" V 4257 3701 40  0000 C CNN
 F 2 "~" V 4180 3700 30  0000 C CNN
@@
 N[0..9]
 $Comp
-L IC_16PIN IC13
+L IC_16PIN IC2
 U 1 1 53FBC5F1
 P 3450 2250
-F 0 "IC13" H 3450 2700 39  0000 C CNN
+F 0 "IC2" H 3450 2700 39  0000 C CNN
 F 1 "IC_16PIN" H 3450 2250 39  0000 C CNN
 F 2 "~" H 3650 1850 60  0000 C CNN
@@
 $EndComp
 $Comp
-L C C14
+L C C6
 U 1 1 53FBC946
-P 2850 2900
-F 0 "C14" H 2850 3000 40  0000 L CNN
-F 1 "C" H 2856 2815 40  0000 L CNN
-F 2 "~" H 2888 2750 30  0000 C CNN
-F 3 "~" H 2850 2900 60  0000 C CNN
-	1    2850 2900
-	1    0    0    -1
+P 3450 1600
+F 0 "C6" H 3450 1700 40  0000 L CNN
+F 1 "0.1u" H 3456 1515 40  0000 L CNN
+F 2 "~" H 3488 1450 30  0000 C CNN
+F 3 "~" H 3450 1600 60  0000 C CNN
+	1    3450 1600
+	0    -1   -1   0
 $EndComp
 $Comp
 L GND #PWR022
 U 1 1 53FBC955
-P 2850 3150
-F 0 "#PWR022" H 2850 3150 30  0001 C CNN
-F 1 "GND" H 2850 3080 30  0001 C CNN
-F 2 "" H 2850 3150 60  0000 C CNN
-F 3 "" H 2850 3150 60  0000 C CNN
-	1    2850 3150
+P 2850 2800
+F 0 "#PWR022" H 2850 2800 30  0001 C CNN
+F 1 "GND" H 2850 2730 30  0001 C CNN
+F 2 "" H 2850 2800 60  0000 C CNN
+F 3 "" H 2850 2800 60  0000 C CNN
+	1    2850 2800
 	1    0    0    -1
 $EndComp
@@
 	2600 2100 3000 2100
 Wire Wire Line
-	2850 1600 2850 2700
+	4000 1450 4000 1900
 Wire Wire Line
 	3000 2400 2850 2400
@@
 	3000 2300 2700 2300
 Wire Wire Line
-	2700 2200 2700 3150
+	2700 2200 2700 2800
 Wire Wire Line
 	3000 2200 2700 2200
@@
 	4000 5900 4350 5900
 Wire Wire Line
-	5350 6300 5350 6800
+	5350 5650 5350 6800
 Wire Wire Line
 	5250 6300 5350 6300
 Wire Wire Line
-	4250 6300 4250 5700
-Wire Wire Line
-	4350 6300 4250 6300
+	4250 5600 4250 6300
+Wire Wire Line
+	4250 6300 4350 6300
 Wire Wire Line
 	2650 6500 4350 6500
@@
 Connection ~ 2700 2600
 Wire Wire Line
-	3900 1900 3900 1700
-Wire Wire Line
-	3900 1700 2850 1700
-Connection ~ 2850 1700
-Wire Wire Line
-	2850 3150 2850 3100
+	2850 1600 2850 2800
 Connection ~ 2850 2400
 Wire Wire Line
@@
 F12 "N[0..9]" I L 7800 2600 60
 $EndSheet
+$Comp
+L C C15
+U 1 1 53FCAC33
+P 4800 5650
+F 0 "C15" H 4800 5750 40  0000 L CNN
+F 1 "0.1u" H 4806 5565 40  0000 L CNN
+F 2 "~" H 4838 5500 30  0000 C CNN
+F 3 "~" H 4800 5650 60  0000 C CNN
+	1    4800 5650
+	0    -1   -1   0
+$EndComp
+Wire Wire Line
+	5350 5650 5000 5650
+Connection ~ 5350 6300
+Wire Wire Line
+	4600 5650 4250 5650
+Connection ~ 4250 5650
+Wire Wire Line
+	4000 1900 3900 1900
+Wire Wire Line
+	3650 1600 4000 1600
+Connection ~ 4000 1600
+Wire Wire Line
+	3250 1600 2850 1600
 $EndSCHEMATC

Commit message: PCB
Connections:
- net labels added: GND_L, L1, L2, L3, L4, L5, L6, L7, L8, PB_P0, PB_P1, PB_P2, PB_P3, PB_P4, PB_P[0..4], PC_P0, PC_P1, PC_P2, PC_P3, PC_P[0..3]
- net labels removed: GND, PB0, PB1, PB2, PB3, PB4, PB[0..4], PC0, PC1, PC2, PC3, PC[0..3]
- wire segments 121 -> 116
Changed lines of the file:
@@
 Sheet 2 13
 Title ""
-Date "30 aug 2014"
+Date "31 aug 2014"
 Rev ""
 Comp ""
@@
 $EndDescr
 Text HLabel 2250 1450 0    60   Input ~ 0
-PB[0..4]
+PB_P[0..4]
 $Comp
 L IC_16PIN IC5
@@
 	2550 6400 2650 6500
 $Comp
-L +5V #PWR015
+L +5V #PWR017
 U 1 1 53F99ADE
 P 4250 5600
-F 0 "#PWR015" H 4250 5690 20  0001 C CNN
+F 0 "#PWR017" H 4250 5690 20  0001 C CNN
 F 1 "+5V" H 4250 5690 30  0000 C CNN
 F 2 "" H 4250 5600 60  0000 C CNN
@@
 	1    0    0    -1
 $EndComp
-$Comp
-L GND #PWR016
-U 1 1 53F99AED
-P 5350 6800
-F 0 "#PWR016" H 5350 6800 30  0001 C CNN
-F 1 "GND" H 5350 6730 30  0001 C CNN
-F 2 "" H 5350 6800 60  0000 C CNN
-F 3 "" H 5350 6800 60  0000 C CNN
-	1    5350 6800
-	1    0    0    -1
-$EndComp
 Entry Wire Line
 	3900 6500 4000 6600
@@
 Entry Wire Line
 	6600 6600 6700 6500
-$Comp
-L GND #PWR017
-U 1 1 53F99C2C
-P 2700 2800
-F 0 "#PWR017" H 2700 2800 30  0001 C CNN
-F 1 "GND" H 2700 2730 30  0001 C CNN
-F 2 "" H 2700 2800 60  0000 C CNN
-F 3 "" H 2700 2800 60  0000 C CNN
-	1    2700 2800
-	1    0    0    -1
-$EndComp
 $Comp
 L +5V #PWR018
@@
 $EndComp
 $Comp
-L GND #PWR020
-U 1 1 53FA3540
-P 5650 5250
-F 0 "#PWR020" H 5650 5250 30  0001 C CNN
-F 1 "GND" H 5650 5180 30  0001 C CNN
-F 2 "" H 5650 5250 60  0000 C CNN
-F 3 "" H 5650 5250 60  0000 C CNN
-	1    5650 5250
-	1    0    0    -1
-$EndComp
-$Comp
 L R R9
 U 1 1 53FA354D
@@
 $EndComp
 $Comp
-L +5V #PWR021
+L +5V #PWR020
 U 1 1 53FAC041
 P 4250 3400
-F 0 "#PWR021" H 4250 3490 20  0001 C CNN
+F 0 "#PWR020" H 4250 3490 20  0001 C CNN
 F 1 "+5V" H 4250 3490 30  0000 C CNN
 F 2 "" H 4250 3400 60  0000 C CNN
@@
 	2500 4450 2600 4550
 Text HLabel 2350 5450 0    60   Input ~ 0
-PC[0..3]
+PC_P[0..3]
 Text Label 2650 1900 0    60   ~ 0
-PB0
+PB_P0
 Text Label 2650 2000 0    60   ~ 0
-PB1
+PB_P1
 Text Label 2650 2100 0    60   ~ 0
-PB2
+PB_P2
 Text Label 2750 6100 0    60   ~ 0
-PC3
+PC_P3
 Text Label 2750 6500 0    60   ~ 0
-PC0
+PC_P0
 Text Label 2750 6400 0    60   ~ 0
-PC1
+PC_P1
 Text Label 2750 6200 0    60   ~ 0
-PC2
+PC_P2
 Text Label 4050 6000 0    60   ~ 0
 N0
@@
 N9
 Text Label 2850 4200 0    60   ~ 0
-PB3
+PB_P3
 Text Label 2850 4550 0    60   ~ 0
-PB4
+PB_P4
 Text Label 7400 2600 0    60   ~ 0
 N[0..9]
@@
 	0    -1   -1   0
 $EndComp
-$Comp
-L GND #PWR022
-U 1 1 53FBC955
-P 2850 2800
-F 0 "#PWR022" H 2850 2800 30  0001 C CNN
-F 1 "GND" H 2850 2730 30  0001 C CNN
-F 2 "" H 2850 2800 60  0000 C CNN
-F 3 "" H 2850 2800 60  0000 C CNN
-	1    2850 2800
-	1    0    0    -1
-$EndComp
 Text GLabel 5650 850  2    60   Input ~ 0
 170V
-$Comp
-L GND #PWR023
-U 1 1 53FBFB0A
-P 5800 5250
-F 0 "#PWR023" H 5800 5250 30  0001 C CNN
-F 1 "GND" H 5800 5180 30  0001 C CNN
-F 2 "" H 5800 5250 60  0000 C CNN
-F 3 "" H 5800 5250 60  0000 C CNN
-	1    5800 5250
-	1    0    0    -1
-$EndComp
 Wire Wire Line
 	4550 850  4550 850
@@
 	3000 2300 2700 2300
 Wire Wire Line
-	2700 2200 2700 2800
+	2700 2200 2700 2850
 Wire Wire Line
 	3000 2200 2700 2200
@@
 	2650 6100 4350 6100
 Wire Wire Line
-	4150 3100 4650 3100
-Wire Wire Line
-	4150 2700 4150 3100
-Wire Wire Line
-	2950 2700 4150 2700
-Wire Wire Line
-	4650 2900 4250 2900
+	4350 3100 4650 3100
+Wire Wire Line
+	2950 2700 4100 2700
+Wire Wire Line
+	4650 2900 4350 2900
 Wire Wire Line
 	4650 2700 4350 2700
 Wire Wire Line
-	4250 2900 4250 2600
-Wire Wire Line
-	4250 2600 3900 2600
-Wire Wire Line
-	4350 2700 4350 2500
-Wire Wire Line
-	4350 2500 3900 2500
-Wire Wire Line
-	4650 2500 4450 2500
-Wire Wire Line
-	4450 2500 4450 2400
-Wire Wire Line
-	4450 2400 3900 2400
-Wire Wire Line
-	4650 2200 4450 2200
-Wire Wire Line
-	4450 2200 4450 2300
-Wire Wire Line
-	4450 2300 3900 2300
-Wire Wire Line
-	3900 2200 4350 2200
-Wire Wire Line
-	4350 2200 4350 2000
+	4100 2600 3900 2600
+Wire Wire Line
+	4100 2500 3900 2500
+Wire Wire Line
+	4650 2500 4350 2500
+Wire Wire Line
+	4100 2400 3900 2400
+Wire Wire Line
+	4650 2200 4350 2200
+Wire Wire Line
+	4100 2300 3900 2300
+Wire Wire Line
+	3900 2200 4100 2200
 Wire Wire Line
 	4350 2000 4650 2000
 Wire Wire Line
-	4650 1800 4250 1800
-Wire Wire Line
-	4250 1800 4250 2100
-Wire Wire Line
-	4250 2100 3900 2100
-Wire Wire Line
-	3900 2000 4150 2000
-Wire Wire Line
-	4150 2000 4150 1600
-Wire Wire Line
-	4150 1600 4650 1600
+	4650 1800 4350 1800
+Wire Wire Line
+	4100 2100 3900 2100
+Wire Wire Line
+	3900 2000 4100 2000
+Wire Wire Line
+	4350 1600 4650 1600
 Wire Wire Line
 	5550 1500 5650 1500
@@
 	6350 2300 7800 2300
 Wire Wire Line
-	5650 5150 5650 5250
+	5650 5150 5650 5300
 Wire Wire Line
 	6150 2100 7800 2100
@@
 Connection ~ 2700 2600
 Wire Wire Line
-	2850 1600 2850 2800
+	2850 1600 2850 2850
 Connection ~ 2850 2400
 Wire Wire Line
@@
 	2950 2500 2950 2700
 Wire Wire Line
-	5800 5150 5800 5250
+	5800 5150 5800 5300
 Wire Wire Line
 	6600 2500 6600 4450
@@
 Wire Wire Line
 	3250 1600 2850 1600
+Text Label 4000 2700 0    60   ~ 0
+L1
+Text Label 4000 2600 0    60   ~ 0
+L2
+Text Label 4000 2500 0    60   ~ 0
+L3
+Text Label 4000 2400 0    60   ~ 0
+L4
+Text Label 4000 2300 0    60   ~ 0
+L5
+Text Label 4000 2200 0    60   ~ 0
+L6
+Text Label 4000 2100 0    60   ~ 0
+L7
+Text Label 4000 2000 0    60   ~ 0
+L8
+Text Label 4350 1600 0    60   ~ 0
+L1
+Text Label 4350 1800 0    60   ~ 0
+L2
+Text Label 4350 2000 0    60   ~ 0
+L3
+Text Label 4350 2200 0    60   ~ 0
+L4
+Text Label 4350 2500 0    60   ~ 0
+L5
+Text Label 4350 2700 0    60   ~ 0
+L6
+Text Label 4350 2900 0    60   ~ 0
+L7
+Text Label 4350 3100 0    60   ~ 0
+L8
+Text GLabel 5250 5300 0    60   Input ~ 0
+GND_L
+Wire Wire Line
+	5800 5300 5250 5300
+Connection ~ 5650 5300
+Text GLabel 5250 6800 0    60   Input ~ 0
+GND_L
+Text GLabel 3000 2850 2    60   Input ~ 0
+GND_L
+Wire Wire Line
+	2700 2850 3000 2850
+Connection ~ 2850 2850
+Wire Wire Line
+	5350 6800 5250 6800
 $EndSCHEMATC
