File: files/pcb/kicad/nixie_tube.sch (KiCad schematic (older format))
At the start: 16 parts, among them K1 CONN_3, K2 CONN_3, K3 CONN_3, K4 CONN_3, U10 NIXIE_IN_16, U11 NIXIE_IN_16, U12 NIXIE_IN_16, U3 NEON, U4 NEON, U5 NEON, U6 NEON, U7 NIXIE_IN_16, U8 NIXIE_IN_16, U9 NIXIE_IN_16

Commit message: 回路図ERC途中
Connections:
- net N7: now reaches U12.11 (8)
- net N7: now also U10.11 (8), U11.11 (8), U7.11 (8), U8.11 (8), U9.11 (8)
- net N8: now reaches U12.12 (9)
- net N8: now also U10.12 (9), U11.12 (9), U7.12 (9), U8.12 (9), U9.12 (9)
- net N9: now reaches U12.13 (0)
- net N9: now also U10.13 (0), U11.13 (0), U7.13 (0), U8.13 (0), U9.13 (0)
- net N0: now reaches U12.2 (1)
- net N0: now also U10.2 (1), U11.2 (1), U7.2 (1), U8.2 (1), U9.2 (1)
- net N1: now reaches U12.3 (7)
- net N1: now also U10.3 (7), U11.3 (7), U7.3 (7), U8.3 (7), U9.3 (7)
- net N2: now reaches U12.4 (3)
- net N2: now also U10.4 (3), U11.4 (3), U7.4 (3), U8.4 (3), U9.4 (3)
- net N3: now reaches U12.6 (4)
- net N3: now also U10.6 (4), U11.6 (4), U7.6 (4), U8.6 (4), U9.6 (4)
- net N4: now reaches U12.7 (5)
- net N4: now also U10.7 (5), U11.7 (5), U7.7 (5), U8.7 (5), U9.7 (5)
- net N5: now reaches U12.8 (6)
- net N5: now also U10.8 (6), U11.8 (6), U7.8 (6), U8.8 (6), U9.8 (6)
- net N6: now reaches U12.9 (2)
- net N6: now also U10.9 (2), U11.9 (2), U7.9 (2), U8.9 (2), U9.9 (2)
Other:
- moved on the sheet: U10, U11, U12, U7, U8, U9

Commit message: 部品リスト・パッケージライブラリを更新
Parts:
- renumbered 200k1 to R30, 200k2 to R31, U3 to U1, U12 to U10, U4 to U2, U5 to U3, U6 to U4, U7 to U5, U8 to U6, U9 to U7, U10 to U8, U11 to U9
Changed lines of the file:
@@
 $EndDescr
 $Comp
-L NIXIE_IN_16 U12
+L NIXIE_IN_16 U10
 U 1 1 53F9F8E3
 P 9250 5850
-F 0 "U12" H 9450 6100 60  0000 C CNN
+F 0 "U10" H 9450 6100 60  0000 C CNN
 F 1 "NIXIE_IN_16" H 8900 6100 60  0000 C CNN
 F 2 "" H 9250 5950 60  0000 C CNN
@@
 	8600 6650 8700 6550
 $Comp
-L NIXIE_IN_16 U9
+L NIXIE_IN_16 U7
 U 1 1 53F9F901
 P 7550 5850
-F 0 "U9" H 7750 6100 60  0000 C CNN
+F 0 "U7" H 7750 6100 60  0000 C CNN
 F 1 "NIXIE_IN_16" H 7200 6100 60  0000 C CNN
 F 2 "" H 7550 5950 60  0000 C CNN
@@
 	6900 6650 7000 6550
 $Comp
-L NIXIE_IN_16 U11
+L NIXIE_IN_16 U9
 U 1 1 53F9F91F
 P 9250 3750
-F 0 "U11" H 9450 4000 60  0000 C CNN
+F 0 "U9" H 9450 4000 60  0000 C CNN
 F 1 "NIXIE_IN_16" H 8900 4000 60  0000 C CNN
 F 2 "" H 9250 3850 60  0000 C CNN
@@
 	8600 4550 8700 4450
 $Comp
-L NIXIE_IN_16 U8
+L NIXIE_IN_16 U6
 U 1 1 53F9F93D
 P 7550 3750
-F 0 "U8" H 7750 4000 60  0000 C CNN
+F 0 "U6" H 7750 4000 60  0000 C CNN
 F 1 "NIXIE_IN_16" H 7200 4000 60  0000 C CNN
 F 2 "" H 7550 3850 60  0000 C CNN
@@
 	6900 4550 7000 4450
 $Comp
-L NIXIE_IN_16 U10
+L NIXIE_IN_16 U8
 U 1 1 53F9F95B
 P 9200 1500
-F 0 "U10" H 9400 1750 60  0000 C CNN
+F 0 "U8" H 9400 1750 60  0000 C CNN
 F 1 "NIXIE_IN_16" H 8850 1750 60  0000 C CNN
 F 2 "" H 9200 1600 60  0000 C CNN
@@
 	8550 2300 8650 2200
 $Comp
-L NIXIE_IN_16 U7
+L NIXIE_IN_16 U5
 U 1 1 53F9F979
 P 7500 1500
-F 0 "U7" H 7700 1750 60  0000 C CNN
+F 0 "U5" H 7700 1750 60  0000 C CNN
 F 1 "NIXIE_IN_16" H 7150 1750 60  0000 C CNN
 F 2 "" H 7500 1600 60  0000 C CNN
@@
 N[0..9]
 $Comp
-L NEON U3
+L NEON U1
 U 1 1 53FA4949
 P 3550 4450
-F 0 "U3" H 3650 4650 60  0000 C CNN
+F 0 "U1" H 3650 4650 60  0000 C CNN
 F 1 "NEON" H 3700 4250 60  0000 C CNN
 F 2 "" H 3650 4650 60  0000 C CNN
@@
 $EndComp
 $Comp
-L NEON U4
+L NEON U2
 U 1 1 53FA4955
 P 3950 4450
-F 0 "U4" H 4050 4650 60  0000 C CNN
+F 0 "U2" H 4050 4650 60  0000 C CNN
 F 1 "NEON" H 4100 4250 60  0000 C CNN
 F 2 "" H 4050 4650 60  0000 C CNN
@@
 $EndComp
 $Comp
-L R 200k1
+L R R30
 U 1 1 53FA4967
 P 3250 5150
-F 0 "200k1" V 3330 5150 40  0000 C CNN
+F 0 "R30" V 3330 5150 40  0000 C CNN
 F 1 "N/A" V 3257 5151 40  0000 C CNN
 F 2 "~" V 3180 5150 30  0000 C CNN
@@
 $EndComp
 $Comp
-L R 200k2
+L R R31
 U 1 1 53FA496D
 P 4350 5150
-F 0 "200k2" V 4430 5150 40  0000 C CNN
+F 0 "R31" V 4430 5150 40  0000 C CNN
 F 1 "N/A" V 4357 5151 40  0000 C CNN
 F 2 "~" V 4280 5150 30  0000 C CNN
@@
 colon_l
 $Comp
-L NEON U5
+L NEON U3
 U 1 1 53FA54C6
 P 4650 4450
-F 0 "U5" H 4750 4650 60  0000 C CNN
+F 0 "U3" H 4750 4650 60  0000 C CNN
 F 1 "NEON" H 4800 4250 60  0000 C CNN
 F 2 "" H 4750 4650 60  0000 C CNN
@@
 $EndComp
 $Comp
-L NEON U6
+L NEON U4
 U 1 1 53FA54CC
 P 5050 4450
-F 0 "U6" H 5150 4650 60  0000 C CNN
+F 0 "U4" H 5150 4650 60  0000 C CNN
 F 1 "NEON" H 5200 4250 60  0000 C CNN
 F 2 "" H 5150 4650 60  0000 C CNN

Commit message: PCB更新
Connections:
- net colon_l: now also R30.1
- net colon_r: now also R31.1
- net at K2.1 (P1), U1.2, U2.2: no longer R30.1
- net at K4.1 (P1), U3.2, U4.2: no longer R31.1
Other:
- moved on the sheet: R30, R31
Changed lines of the file:
@@
 Sheet 3 13
 Title ""
-Date "28 aug 2014"
+Date "30 aug 2014"
 Rev ""
 Comp ""
@@
 L R R30
 U 1 1 53FA4967
-P 3250 5150
-F 0 "R30" V 3330 5150 40  0000 C CNN
-F 1 "N/A" V 3257 5151 40  0000 C CNN
-F 2 "~" V 3180 5150 30  0000 C CNN
-F 3 "~" H 3250 5150 30  0000 C CNN
-	1    3250 5150
+P 2800 4000
+F 0 "R30" V 2880 4000 40  0000 C CNN
+F 1 "N/A" V 2807 4001 40  0000 C CNN
+F 2 "~" V 2730 4000 30  0000 C CNN
+F 3 "~" H 2800 4000 30  0000 C CNN
+	1    2800 4000
 	1    0    0    -1
 $EndComp
@@
 L R R31
 U 1 1 53FA496D
-P 4350 5150
-F 0 "R31" V 4430 5150 40  0000 C CNN
-F 1 "N/A" V 4357 5151 40  0000 C CNN
-F 2 "~" V 4280 5150 30  0000 C CNN
-F 3 "~" H 4350 5150 30  0000 C CNN
-	1    4350 5150
+P 3000 4100
+F 0 "R31" V 3080 4100 40  0000 C CNN
+F 1 "N/A" V 3007 4101 40  0000 C CNN
+F 2 "~" V 2930 4100 30  0000 C CNN
+F 3 "~" H 3000 4100 30  0000 C CNN
+	1    3000 4100
 	1    0    0    -1
 $EndComp
@@
 	3250 4850 3950 4850
 Wire Wire Line
-	3250 3900 3250 4900
+	2800 2750 2800 3750
 Wire Wire Line
 	3550 4800 3550 4850
@@
 	4350 4850 5050 4850
 Wire Wire Line
-	4350 3900 4350 4900
+	3000 2850 3000 3850
 Wire Wire Line
 	4650 4800 4650 4850
@@
 L GND #PWR024
 U 1 1 53FB424E
-P 3250 5500
-F 0 "#PWR024" H 3250 5500 30  0001 C CNN
-F 1 "GND" H 3250 5430 30  0001 C CNN
-F 2 "" H 3250 5500 60  0000 C CNN
-F 3 "" H 3250 5500 60  0000 C CNN
-	1    3250 5500
+P 2800 4350
+F 0 "#PWR024" H 2800 4350 30  0001 C CNN
+F 1 "GND" H 2800 4280 30  0001 C CNN
+F 2 "" H 2800 4350 60  0000 C CNN
+F 3 "" H 2800 4350 60  0000 C CNN
+	1    2800 4350
 	1    0    0    -1
 $EndComp
@@
 L GND #PWR025
 U 1 1 53FB425D
-P 4350 5500
-F 0 "#PWR025" H 4350 5500 30  0001 C CNN
-F 1 "GND" H 4350 5430 30  0001 C CNN
-F 2 "" H 4350 5500 60  0000 C CNN
-F 3 "" H 4350 5500 60  0000 C CNN
-	1    4350 5500
-	1    0    0    -1
-$EndComp
-Wire Wire Line
-	3250 5500 3250 5400
-Wire Wire Line
-	4350 5500 4350 5400
-Connection ~ 4350 4850
-Connection ~ 3250 4850
+P 3000 4450
+F 0 "#PWR025" H 3000 4450 30  0001 C CNN
+F 1 "GND" H 3000 4380 30  0001 C CNN
+F 2 "" H 3000 4450 60  0000 C CNN
+F 3 "" H 3000 4450 60  0000 C CNN
+	1    3000 4450
+	1    0    0    -1
+$EndComp
+Wire Wire Line
+	2800 4350 2800 4250
+Wire Wire Line
+	3000 4450 3000 4350
 Text Label 6950 2150 1    60   ~ 0
 N0
@@
 Text Label 8100 6500 1    60   ~ 0
 N9
+Wire Wire Line
+	4350 4850 4350 3900
+Wire Wire Line
+	3250 4850 3250 3900
+Connection ~ 3000 2850
+Connection ~ 2800 2750
 $EndSCHEMATC

Commit message: PCB
Connections:
- net GND renamed GND_L

Commit message: 設計見直し
部品見直し
USB・DCジャック自動切り替え
マイコンを下段のボードに移動
ニキシー管駆動電源を上段ボードに移動
Connections:
- net GND_L renamed GND
Changed lines of the file:
@@
 $Descr A4 11693 8268
 encoding utf-8
-Sheet 3 11
+Sheet 3 8
 Title ""
-Date "31 aug 2014"
+Date "1 sep 2014"
 Rev ""
 Comp ""
@@
 Text Label 8100 6500 1    60   ~ 0
 N9
-Text GLabel 2600 4600 0    60   Input ~ 0
-GND_L
 Wire Wire Line
 	8700 6550 8700 6350
@@
 Connection ~ 2800 2750
 Wire Wire Line
-	3000 4600 2600 4600
-Wire Wire Line
 	2800 4250 2800 4600
-Connection ~ 2800 4600
+$Comp
+L GND #PWR027
+U 1 1 5404E81E
+P 2800 4600
+F 0 "#PWR027" H 2800 4600 30  0001 C CNN
+F 1 "GND" H 2800 4530 30  0001 C CNN
+F 2 "" H 2800 4600 60  0000 C CNN
+F 3 "" H 2800 4600 60  0000 C CNN
+	1    2800 4600
+	1    0    0    -1
+$EndComp
+$Comp
+L GND #PWR028
+U 1 1 5404E82D
+P 3000 4600
+F 0 "#PWR028" H 3000 4600 30  0001 C CNN
+F 1 "GND" H 3000 4530 30  0001 C CNN
+F 2 "" H 3000 4600 60  0000 C CNN
+F 3 "" H 3000 4600 60  0000 C CNN
+	1    3000 4600
+	1    0    0    -1
+$EndComp
 $EndSCHEMATC
