File: files/pcb/kicad/nixie_tube.sch (KiCad schematic (older format))
At the start: 16 parts, among them K1 CONN_3, K2 CONN_3, K3 CONN_3, K4 CONN_3, U1 NEON, U10 NIXIE_IN_16, U2 NEON, U3 NEON, U4 NEON, U5 NIXIE_IN_16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

Commit message: 基板が描けた
Connections:
- net NEL1: now reaches K2.2 (PM), U1.1
- net NEG1: now reaches K2.1 (P1), U1.2, U2.2
- net NEU1: now reaches K2.3 (P3), U2.1
- net NEL2: now reaches K4.2 (PM), U3.1
- net NEG2: now reaches K4.1 (P1), U3.2, U4.2
- net NEU2: now reaches K4.3 (P3), U4.1
Changed lines of the file:
@@
 Sheet 3 8
 Title ""
-Date "4 sep 2014"
+Date "5 sep 2014"
 Rev ""
 Comp ""
@@
 	2800 4250 2800 4600
 $Comp
-L GND #PWR028
+L GND #PWR019
 U 1 1 5404E81E
 P 2800 4600
-F 0 "#PWR028" H 2800 4600 30  0001 C CNN
+F 0 "#PWR019" H 2800 4600 30  0001 C CNN
 F 1 "GND" H 2800 4530 30  0001 C CNN
 F 2 "" H 2800 4600 60  0000 C CNN
@@
 $EndComp
 $Comp
-L GND #PWR029
+L GND #PWR020
 U 1 1 5404E82D
 P 3000 4600
-F 0 "#PWR029" H 3000 4600 30  0001 C CNN
+F 0 "#PWR020" H 3000 4600 30  0001 C CNN
 F 1 "GND" H 3000 4530 30  0001 C CNN
 F 2 "" H 3000 4600 60  0000 C CNN
@@
 	1    0    0    -1
 $EndComp
+Text Label 4850 3950 0    60   ~ 0
+NEU2
+Text Label 4600 4050 0    60   ~ 0
+NEL2
+Text Label 4400 4850 0    60   ~ 0
+NEG2
+Text Label 3300 4850 0    60   ~ 0
+NEG1
+Text Label 3500 4050 0    60   ~ 0
+NEL1
+Text Label 3700 3950 0    60   ~ 0
+NEU1
 $EndSCHEMATC
