File: files/pcb/kicad/power.sch (KiCad schematic (older format))
At the start: 27 parts, among them IC10 FET, IC8 MY_3_TERMINAL_REGULATOR, IC9 ICM7555CD, T1 2SC, T2 2SC, T3 2SA, U11 DC_JACK

Commit message: 設計見直し
部品見直し
USB・DCジャック自動切り替え
マイコンを下段のボードに移動
ニキシー管駆動電源を上段ボードに移動
Parts:
- removed IC10: FET, symbol FET
- removed T2: 2SC, TO92, symbol 2SC
- removed T3: 2SA, TO92, symbol 2SA
- added D6, D7: DIODE, ~, symbol DIODE
- added IC10: MY_FET_P, ~, symbol MY_FET_P
- added IC12: MY_NPN, symbol MY_NPN
- added IC13: MY_PNP, symbol MY_PNP
- added IC14: MY_FET_N, ~, symbol MY_FET_N
Connections:
- net labels added: PIN9V, PINGND, USB5V
- net labels removed: 5V_L, GND_L
- wire segments 82 -> 80
Other:
- moved on the sheet: C10, C11, C12, C13, C7, C8, C9, D2, F1, IC9, L1, R12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

Commit message: PCB更新
ニキシー管の足を接続
電源仮接続
Connections:
- wire segments 80 -> 81
Other:
- moved on the sheet: C11, C7, C8, C9, D6, D7, F1, U11
Changed lines of the file:
@@
 Sheet 5 8
 Title ""
-Date "1 sep 2014"
+Date "2 sep 2014"
 Rev ""
 Comp ""
@@
 L C C8
 U 1 1 53F8BD8A
-P 6150 2300
-F 0 "C8" H 6150 2400 40  0000 L CNN
-F 1 "0.1u" H 6150 2200 40  0000 L CNN
-F 2 "~" H 6188 2150 30  0000 C CNN
-F 3 "~" H 6150 2300 60  0000 C CNN
-	1    6150 2300
+P 4200 2350
+F 0 "C8" H 4200 2450 40  0000 L CNN
+F 1 "0.1u" H 4200 2250 40  0000 L CNN
+F 2 "~" H 4238 2200 30  0000 C CNN
+F 3 "~" H 4200 2350 60  0000 C CNN
+	1    4200 2350
 	1    0    0    -1
 $EndComp
@@
 L C C7
 U 1 1 53F8BD97
-P 5800 2300
-F 0 "C7" H 5800 2400 40  0000 L CNN
-F 1 "25V 10u" H 5800 2200 40  0000 L CNN
-F 2 "~" H 5838 2150 30  0000 C CNN
-F 3 "~" H 5800 2300 60  0000 C CNN
-	1    5800 2300
+P 3850 2350
+F 0 "C7" H 3850 2450 40  0000 L CNN
+F 1 "25V 10u" H 3850 2250 40  0000 L CNN
+F 2 "~" H 3888 2200 30  0000 C CNN
+F 3 "~" H 3850 2350 60  0000 C CNN
+	1    3850 2350
 	1    0    0    -1
 $EndComp
@@
 L C C11
 U 1 1 53F8BD9D
-P 7350 2200
-F 0 "C11" H 7350 2300 40  0000 L CNN
-F 1 "25V 10u" H 7350 2100 40  0000 L CNN
-F 2 "~" H 7388 2050 30  0000 C CNN
-F 3 "~" H 7350 2200 60  0000 C CNN
-	1    7350 2200
+P 6200 2250
+F 0 "C11" H 6200 2350 40  0000 L CNN
+F 1 "25V 10u" H 6200 2150 40  0000 L CNN
+F 2 "~" H 6238 2100 30  0000 C CNN
+F 3 "~" H 6200 2250 60  0000 C CNN
+	1    6200 2250
 	1    0    0    -1
 $EndComp
@@
 L C C9
 U 1 1 53F8BDA3
-P 7050 2200
-F 0 "C9" H 7050 2300 40  0000 L CNN
-F 1 "0.1u" H 7050 2100 40  0000 L CNN
-F 2 "~" H 7088 2050 30  0000 C CNN
-F 3 "~" H 7050 2200 60  0000 C CNN
-	1    7050 2200
+P 5100 2250
+F 0 "C9" H 5100 2350 40  0000 L CNN
+F 1 "0.1u" H 5100 2150 40  0000 L CNN
+F 2 "~" H 5138 2100 30  0000 C CNN
+F 3 "~" H 5100 2250 60  0000 C CNN
+	1    5100 2250
 	1    0    0    -1
 $EndComp
@@
 L FUSE F1
 U 1 1 53F8C1A7
-P 5450 1950
-F 0 "F1" H 5550 2000 40  0000 C CNN
-F 1 "FUSE" H 5350 1900 40  0000 C CNN
-F 2 "~" H 5450 1950 60  0000 C CNN
-F 3 "~" H 5450 1950 60  0000 C CNN
-	1    5450 1950
+P 3500 2000
+F 0 "F1" H 3600 2050 40  0000 C CNN
+F 1 "FUSE" H 3400 1950 40  0000 C CNN
+F 2 "~" H 3500 2000 60  0000 C CNN
+F 3 "~" H 3500 2000 60  0000 C CNN
+	1    3500 2000
 	1    0    0    -1
 $EndComp
@@
 L DC_JACK U11
 U 1 1 53FB6A7A
-P 3650 2550
-F 0 "U11" H 3500 2725 60  0000 C CNN
-F 1 "DC_JACK" H 3650 2375 60  0000 C CNN
-F 2 "" H 3500 2725 60  0000 C CNN
-F 3 "" H 3500 2725 60  0000 C CNN
-	1    3650 2550
+P 2700 2100
+F 0 "U11" H 2550 2275 60  0000 C CNN
+F 1 "DC_JACK" H 2700 1925 60  0000 C CNN
+F 2 "" H 2550 2275 60  0000 C CNN
+F 3 "" H 2550 2275 60  0000 C CNN
+	1    2700 2100
 	1    0    0    -1
 $EndComp
@@
 L +9V #PWR029
 U 1 1 53FCA114
-P 5200 1850
-F 0 "#PWR029" H 5200 1820 20  0001 C CNN
-F 1 "+9V" H 5200 1960 30  0000 C CNN
-F 2 "" H 5200 1850 60  0000 C CNN
-F 3 "" H 5200 1850 60  0000 C CNN
-	1    5200 1850
+P 3250 1900
+F 0 "#PWR029" H 3250 1870 20  0001 C CNN
+F 1 "+9V" H 3250 2010 30  0000 C CNN
+F 2 "" H 3250 1900 60  0000 C CNN
+F 3 "" H 3250 1900 60  0000 C CNN
+	1    3250 1900
 	1    0    0    -1
 $EndComp
@@
 L MY_3_TERMINAL_REGULATOR IC8
 U 1 1 53FF5CD5
-P 6600 2000
-F 0 "IC8" H 6750 1804 60  0000 C CNN
-F 1 "MY_3_TERMINAL_REGULATOR" H 6600 2200 60  0000 C CNN
-F 2 "~" H 6600 2000 60  0000 C CNN
-F 3 "~" H 6600 2000 60  0000 C CNN
-	1    6600 2000
+P 4650 2050
+F 0 "IC8" H 4800 1854 60  0000 C CNN
+F 1 "MY_3_TERMINAL_REGULATOR" H 4650 2250 60  0000 C CNN
+F 2 "~" H 4650 2050 60  0000 C CNN
+F 3 "~" H 4650 2050 60  0000 C CNN
+	1    4650 2050
 	1    0    0    -1
 $EndComp
@@
 	5650 4950 5650 5500
 Wire Wire Line
-	6600 2650 6600 2250
-Wire Wire Line
-	7000 1950 7550 1950
-Wire Wire Line
-	7050 1950 7050 2000
-Wire Wire Line
-	7350 1950 7350 2000
-Connection ~ 7050 1950
-Wire Wire Line
-	5700 1950 6200 1950
-Wire Wire Line
-	6150 1950 6150 2100
-Connection ~ 6150 1950
-Wire Wire Line
-	7050 2650 7050 2400
-Wire Wire Line
-	7350 2650 7350 2400
-Wire Wire Line
-	6150 2650 6150 2500
-Wire Wire Line
-	7550 1950 7550 1850
-Connection ~ 7350 1950
-Wire Wire Line
-	5800 2100 5800 1950
-Connection ~ 5800 1950
+	4650 2700 4650 2300
+Wire Wire Line
+	5050 2000 5650 2000
+Wire Wire Line
+	6050 2000 6550 2000
+Wire Wire Line
+	5100 2000 5100 2050
+Wire Wire Line
+	6200 1300 6200 2050
+Connection ~ 5100 2000
+Wire Wire Line
+	3750 2000 4250 2000
+Wire Wire Line
+	4200 2000 4200 2150
+Connection ~ 4200 2000
+Wire Wire Line
+	5100 2700 5100 2450
+Wire Wire Line
+	6200 2700 6200 2450
+Wire Wire Line
+	4200 2700 4200 2550
+Wire Wire Line
+	6550 2000 6550 1900
+Connection ~ 6200 2000
+Wire Wire Line
+	3850 2150 3850 2000
+Connection ~ 3850 2000
 Connection ~ 4900 4950
 Wire Wire Line
@@
 Connection ~ 4300 3900
 Wire Wire Line
-	4000 2650 7550 2650
+	3050 2200 3050 2700
+Wire Wire Line
+	3050 2700 6550 2700
 Wire Wire Line
 	8850 6350 8850 4800
 Wire Wire Line
 	5100 6350 5100 5350
-Connection ~ 5200 1950
+Connection ~ 3250 2000
 Wire Wire Line
 	7150 1350 7150 1400
@@
 Wire Wire Line
 	6900 1400 6900 1350
-Connection ~ 7050 2650
-Connection ~ 6600 2650
-Connection ~ 6150 2650
+Connection ~ 5100 2700
+Connection ~ 4650 2700
+Connection ~ 4200 2700
 Wire Wire Line
 	2550 6350 8850 6350
@@
 Wire Wire Line
 	3550 3900 3550 4150
-Text GLabel 4000 1950 0    60   Input ~ 0
+Text GLabel 3050 1300 0    60   Input ~ 0
 USB5V
 $Comp
 L DIODE D6
 U 1 1 5404BD97
-P 4800 1950
-F 0 "D6" H 4800 2050 40  0000 C CNN
-F 1 "DIODE" H 4800 1850 40  0000 C CNN
-F 2 "~" H 4800 1950 60  0000 C CNN
-F 3 "~" H 4800 1950 60  0000 C CNN
-	1    4800 1950
+P 5850 1300
+F 0 "D6" H 5850 1400 40  0000 C CNN
+F 1 "DIODE" H 5850 1200 40  0000 C CNN
+F 2 "~" H 5850 1300 60  0000 C CNN
+F 3 "~" H 5850 1300 60  0000 C CNN
+	1    5850 1300
 	1    0    0    -1
 $EndComp
@@
 L DIODE D7
 U 1 1 5404BDA6
-P 5000 2150
-F 0 "D7" H 5000 2250 40  0000 C CNN
-F 1 "DIODE" H 5000 2050 40  0000 C CNN
-F 2 "~" H 5000 2150 60  0000 C CNN
-F 3 "~" H 5000 2150 60  0000 C CNN
-	1    5000 2150
-	0    -1   -1   0
-$EndComp
-Wire Wire Line
-	5000 1950 5200 1950
-Wire Wire Line
-	4000 2450 5000 2450
-NoConn ~ 4000 2550
-Wire Wire Line
-	4250 1950 4000 1950
-Wire Wire Line
-	4400 2150 4400 2450
-Connection ~ 4400 2450
-Wire Wire Line
-	5200 1950 5200 1850
+P 5850 2000
+F 0 "D7" H 5850 2100 40  0000 C CNN
+F 1 "DIODE" H 5850 1900 40  0000 C CNN
+F 2 "~" H 5850 2000 60  0000 C CNN
+F 3 "~" H 5850 2000 60  0000 C CNN
+	1    5850 2000
+	1    0    0    -1
+$EndComp
+Wire Wire Line
+	6050 1300 6200 1300
+Wire Wire Line
+	3050 2000 3250 2000
+NoConn ~ 3050 2100
+Wire Wire Line
+	5200 1300 3050 1300
+Wire Wire Line
+	5350 1500 5350 2000
+Wire Wire Line
+	3250 2000 3250 1900
 $Comp
 L GND #PWR034
 U 1 1 5404CB58
-P 7550 2750
-F 0 "#PWR034" H 7550 2750 30  0001 C CNN
-F 1 "GND" H 7550 2680 30  0001 C CNN
-F 2 "" H 7550 2750 60  0000 C CNN
-F 3 "" H 7550 2750 60  0000 C CNN
-	1    7550 2750
-	1    0    0    -1
-$EndComp
-Wire Wire Line
-	5800 2500 5800 2650
-Connection ~ 5800 2650
-Wire Wire Line
-	7550 2650 7550 2750
-Connection ~ 7350 2650
+P 6550 2800
+F 0 "#PWR034" H 6550 2800 30  0001 C CNN
+F 1 "GND" H 6550 2730 30  0001 C CNN
+F 2 "" H 6550 2800 60  0000 C CNN
+F 3 "" H 6550 2800 60  0000 C CNN
+	1    6550 2800
+	1    0    0    -1
+$EndComp
+Wire Wire Line
+	3850 2550 3850 2700
+Connection ~ 3850 2700
+Wire Wire Line
+	6550 2700 6550 2800
+Connection ~ 6200 2700
 Wire Wire Line
 	2950 4150 2950 6350
@@
 Text GLabel 2550 3400 0    60   Input ~ 0
 PIN9V
-Wire Wire Line
-	5000 2450 5000 2350
 $Comp
 L MY_FET_P IC10
 U 1 1 5404BB69
-P 4400 1950
-F 0 "IC10" H 4250 2100 60  0000 C CNN
-F 1 "MY_FET_P" H 4175 1800 60  0000 C CNN
-F 2 "~" H 4250 2100 60  0000 C CNN
-F 3 "~" H 4250 2100 60  0000 C CNN
-	1    4400 1950
+P 5350 1300
+F 0 "IC10" V 5600 1300 60  0000 C CNN
+F 1 "MY_FET_P" V 5500 1300 60  0000 C CNN
+F 2 "~" H 5200 1450 60  0000 C CNN
+F 3 "~" H 5200 1450 60  0000 C CNN
+	1    5350 1300
 	0    1    -1   0
 $EndComp
 Wire Wire Line
-	4550 1950 4600 1950
+	5500 1300 5650 1300
 $Comp
 L MY_FET_N IC14
@@
 L +5V #PWR035
 U 1 1 540509DD
-P 7550 1850
-F 0 "#PWR035" H 7550 1940 20  0001 C CNN
-F 1 "+5V" H 7550 1940 30  0000 C CNN
-F 2 "" H 7550 1850 60  0000 C CNN
-F 3 "" H 7550 1850 60  0000 C CNN
-	1    7550 1850
-	1    0    0    -1
-$EndComp
+P 6550 1900
+F 0 "#PWR035" H 6550 1990 20  0001 C CNN
+F 1 "+5V" H 6550 1990 30  0000 C CNN
+F 2 "" H 6550 1900 60  0000 C CNN
+F 3 "" H 6550 1900 60  0000 C CNN
+	1    6550 1900
+	1    0    0    -1
+$EndComp
+Connection ~ 5350 2000
 $EndSCHEMATC

Commit message: PCB更新
Parts:
- added R33: R, ~, symbol R
Connections:
- wire segments 81 -> 82
Changed lines of the file:
@@
 Sheet 5 8
 Title ""
-Date "2 sep 2014"
+Date "4 sep 2014"
 Rev ""
 Comp ""
@@
 170V
 $Comp
-L +9V #PWR029
+L +9V #PWR030
 U 1 1 53FCA114
 P 3250 1900
-F 0 "#PWR029" H 3250 1870 20  0001 C CNN
+F 0 "#PWR030" H 3250 1870 20  0001 C CNN
 F 1 "+9V" H 3250 2010 30  0000 C CNN
 F 2 "" H 3250 1900 60  0000 C CNN
@@
 $EndComp
 $Comp
-L +9V #PWR030
+L +9V #PWR031
 U 1 1 53FC9A5B
 P 6750 1350
-F 0 "#PWR030" H 6750 1320 20  0001 C CNN
+F 0 "#PWR031" H 6750 1320 20  0001 C CNN
 F 1 "+9V" H 6750 1460 30  0000 C CNN
 F 2 "" H 6750 1350 60  0000 C CNN
@@
 $EndComp
 $Comp
-L PWR_FLAG #FLG031
+L PWR_FLAG #FLG032
 U 1 1 53FC9A79
 P 7150 1350
-F 0 "#FLG031" H 7150 1445 30  0001 C CNN
+F 0 "#FLG032" H 7150 1445 30  0001 C CNN
 F 1 "PWR_FLAG" H 7150 1530 30  0000 C CNN
 F 2 "" H 7150 1350 60  0000 C CNN
@@
 $EndComp
 $Comp
-L PWR_FLAG #FLG032
+L PWR_FLAG #FLG033
 U 1 1 53FC9AFB
 P 6900 1350
-F 0 "#FLG032" H 6900 1445 30  0001 C CNN
+F 0 "#FLG033" H 6900 1445 30  0001 C CNN
 F 1 "PWR_FLAG" H 6900 1530 30  0000 C CNN
 F 2 "" H 6900 1350 60  0000 C CNN
@@
 	6950 3400 6950 3450
 Connection ~ 5100 3400
-Wire Wire Line
-	6950 6350 6950 5750
 Connection ~ 6950 3400
 Wire Wire Line
@@
 	5050 2000 5650 2000
 Wire Wire Line
-	6050 2000 6550 2000
+	6050 2000 6750 2000
 Wire Wire Line
 	5100 2000 5100 2050
@@
 Connection ~ 5100 6350
 $Comp
-L GND #PWR033
+L GND #PWR034
 U 1 1 53FC9AEE
 P 7150 1400
-F 0 "#PWR033" H 7150 1400 30  0001 C CNN
+F 0 "#PWR034" H 7150 1400 30  0001 C CNN
 F 1 "GND" H 7150 1330 30  0001 C CNN
 F 2 "" H 7150 1400 60  0000 C CNN
@@
 	3250 2000 3250 1900
 $Comp
-L GND #PWR034
+L GND #PWR035
 U 1 1 5404CB58
 P 6550 2800
-F 0 "#PWR034" H 6550 2800 30  0001 C CNN
+F 0 "#PWR035" H 6550 2800 30  0001 C CNN
 F 1 "GND" H 6550 2730 30  0001 C CNN
 F 2 "" H 6550 2800 60  0000 C CNN
@@
 $EndComp
 $Comp
-L +5V #PWR035
+L +5V #PWR036
 U 1 1 540509DD
 P 6550 1900
-F 0 "#PWR035" H 6550 1990 20  0001 C CNN
+F 0 "#PWR036" H 6550 1990 20  0001 C CNN
 F 1 "+5V" H 6550 1990 30  0000 C CNN
 F 2 "" H 6550 1900 60  0000 C CNN
@@
 $EndComp
 Connection ~ 5350 2000
+$Comp
+L R R33
+U 1 1 54087537
+P 6950 6000
+F 0 "R33" V 7030 6000 40  0000 C CNN
+F 1 "R" V 6957 6001 40  0000 C CNN
+F 2 "~" V 6880 6000 30  0000 C CNN
+F 3 "~" H 6950 6000 30  0000 C CNN
+	1    6950 6000
+	1    0    0    -1
+$EndComp
+Wire Wire Line
+	6950 6350 6950 6250
+$Comp
+L PWR_FLAG #FLG037
+U 1 1 54087A33
+P 6750 1900
+F 0 "#FLG037" H 6750 1995 30  0001 C CNN
+F 1 "PWR_FLAG" H 6750 2080 30  0000 C CNN
+F 2 "" H 6750 1900 60  0000 C CNN
+F 3 "" H 6750 1900 60  0000 C CNN
+	1    6750 1900
+	1    0    0    -1
+$EndComp
+Wire Wire Line
+	6750 2000 6750 1900
+Connection ~ 6550 2000
 $EndSCHEMATC
