File: files/circuit/kicad/kicad_project.kicad_pcb (KiCad board)
At the start: 2 copper layers, 100 x 90 mm, 113 parts, among them CON1 USB_MINI_B, IC1 ATMEGA328-A, IC10 MY_FET_P, IC11 DS1307, IC12 MY_NPN, IC13 MY_PNP, IC14 MY_FET_N, IC2 74LC138, IC3 TLP627, IC4 TLP627, IC5 SN74141_K155NA, IC6 TLP627-4, IC7 TLP627-4, IC8 MY_3_TERMINAL_REGULATOR, IC9 ICM7555CD, K1 CONN_3, K3 CONN_3, K4 CONN_3, K5 CONN_3, P1 CONN_6, SW3 SW_PUSH, SW4 SW_PUSH, SW5 SW_PUSH, T1 2SC, U10 NIXIE_IN_16, U11 DC_JACK, U12 MY_PIN72, U13 MY_PIN72, U14 NEON, U15 MY_PIN52, U16 MY_PIN52, U17 MY_PIN52, U18 MY_PIN52, U19 NEON, U3 NEON, U4 NEON, U5 NIXIE_IN_16, U6 NIXIE_IN_16, U7 NIXIE_IN_16, U8 NIXIE_IN_16, U9 NIXIE_IN_16, X1 12MHz, X2 32.768kHz

Commit message: 配線の太さを調整
Routing:
- net PINGND: track 395.4 -> 453.3 mm
- net +5V: track 147.1 -> 202.0 mm
- net N-0000052: track 63.0 -> 108.2 mm
- net PIN9V: track 132.4 -> 171.7 mm
- net GND: track 457.2 -> 485.1 mm
- net N-0000079: track 22.2 -> 49.2 mm
- net 170V: track 14.2 -> 30.7 mm
- net +9V: track 21.9 -> 30.8 mm
- net N-0000074: track 13.3 -> 20.5 mm
- net N-0000081: track 14.2 -> 20.1 mm
- net N-0000071: track 9.38 -> 14.4 mm
- net PIN170V: track 2.86 -> 5.82 mm
- net N-0000082: track 17.4 -> 20.2 mm
- net N-0000072: track 5.03 -> 7.48 mm
- net N-0000080: track 2.01 -> 4.15 mm
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
Commit message: 基板完成、発注版
Parts:
- removed U10, U5, U6, U7, U8, U9: NIXIE_IN_16, my_nixie
- added NI1: NIXIE_IN_16, my_nixie, F.Cu at (112.0, 143.5)
- added NI2: NIXIE_IN_16, my_nixie, F.Cu at (125.5, 143.5)
- added NI3: NIXIE_IN_16, my_nixie, F.Cu at (143.2, 143.5)
- added NI4: NIXIE_IN_16, my_nixie, F.Cu at (156.8, 143.5)
- added NI5: NIXIE_IN_16, my_nixie, F.Cu at (174.5, 143.5)
- added NI6: NIXIE_IN_16, my_nixie, F.Cu at (188.0, 143.5)
- K2: value (none) -> CONN_3
- U1, U2: value (none) -> NEON
Connections:
- IC5 pad 1: /nixie/N1 -> /nixie/N8
- IC5 pad 10: /nixie/N7 -> /nixie/N4
- IC5 pad 11: /nixie/N8 -> /nixie/N5
- IC5 pad 13: /nixie/N4 -> /nixie/N6
- IC5 pad 14: /nixie/N5 -> /nixie/N1
- IC5 pad 15: /nixie/N2 -> /nixie/N0
- IC5 pad 16: /nixie/N3 -> /nixie/N7
- IC5 pad 2: /nixie/N0 -> /nixie/N9
- IC5 pad 8: /nixie/N9 -> /nixie/N2
- IC5 pad 9: /nixie/N6 -> /nixie/N3
- U15 pad 1: PIN5V -> PINGND
- U15 pad 10: PINGND -> PIN5V
- U15 pad 4: PIN9V -> PINGND
- U15 pad 6: PINGND -> PIN9V
- U16 pad 1: +5V -> GND
- U16 pad 10: GND -> +5V
- U16 pad 4: +9V -> GND
- U16 pad 6: GND -> +9V
Routing:
- net +5V: track 202.0 -> 156.3 mm
- net /nixie/N1: track 129.1 -> 97.8 mm, vias 1 -> 0
- net /nixie/N0: track 127.0 -> 99.6 mm, vias 1 -> 0
- net PIN9V: track 171.7 -> 145.3 mm
- net PIN5V: track 136.2 -> 154.1 mm
- net /nixie/Sheet53F9F7BA/dot_cathode_r: track 124.8 -> 137.0 mm
- net GND: track 485.1 -> 496.3 mm
- net /nixie/N4: track 99.7 -> 110.3 mm
- net /nixie/N9: track 116.2 -> 106.0 mm, vias 0 -> 1
- net /nixie/Sheet53F9F7BA/dot_cathode_l: track 112.9 -> 122.2 mm
- net PINGND: track 453.3 -> 445.6 mm
- net /nixie/N6: track 97.9 -> 105.0 mm
- net /nixie/N3: track 102.9 -> 107.2 mm, vias 1 -> 0
- net /nixie/N2: track 107.8 -> 111.6 mm, vias 1 -> 0
- net /nixie/Sheet53F9F7BA/colon_r: track 44.5 -> 41.0 mm
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- added copper zone on B.Cu, net (none)
- added copper zone on F.Cu, net (none)
