File: files/circuit/kicad/kicad_project.sch (KiCad schematic (older format))
At the start: 20 parts, among them IC1 ATMEGA328-A, P1 CONN_6, U12 MY_PIN72, U13 MY_PIN72, U15 MY_PIN52, U16 MY_PIN52, U17 MY_PIN52, U18 MY_PIN52, X1 12MHz

Commit message: 回路完成、ディレクトリ構造変更
Connections:
- wire segments 83 -> 82
Changed lines of the file:
@@
 Sheet 1 8
 Title ""
-Date "6 sep 2014"
+Date "7 sep 2014"
 Rev ""
 Comp ""
@@
 	9600 6500 9650 6500
 Wire Wire Line
-	5900 6800 5900 6600
+	5900 6300 5900 6800
 Wire Wire Line
 	1850 5500 1350 5500
@@
 	6650 6750 5900 6750
 Connection ~ 5900 6750
-Wire Wire Line
-	5900 6300 5900 6400
 Wire Wire Line
 	5800 6400 5800 6700
@@
 Connection ~ 9650 6100
 Connection ~ 9650 6300
+Connection ~ 5900 6600
 $EndSCHEMATC

Commit message: 基板完成、発注版
Connections:
- wire segments 82 -> 73
Changed lines of the file:
@@
 Sheet 1 8
 Title ""
-Date "7 sep 2014"
+Date "8 sep 2014"
 Rev ""
 Comp ""
@@
 L +5V #PWR01
 U 1 1 54045B6C
-P 5900 6200
-F 0 "#PWR01" H 5900 6290 20  0001 C CNN
-F 1 "+5V" H 5900 6290 30  0000 C CNN
-F 2 "" H 5900 6200 60  0000 C CNN
-F 3 "" H 5900 6200 60  0000 C CNN
-	1    5900 6200
+P 6650 6200
+F 0 "#PWR01" H 6650 6290 20  0001 C CNN
+F 1 "+5V" H 6650 6290 30  0000 C CNN
+F 2 "" H 6650 6200 60  0000 C CNN
+F 3 "" H 6650 6200 60  0000 C CNN
+	1    6650 6200
 	1    0    0    -1
 $EndComp
@@
 L +9V #PWR04
 U 1 1 5408AC70
-P 5550 6400
-F 0 "#PWR04" H 5550 6370 20  0001 C CNN
-F 1 "+9V" H 5550 6510 30  0000 C CNN
-F 2 "" H 5550 6400 60  0000 C CNN
-F 3 "" H 5550 6400 60  0000 C CNN
-	1    5550 6400
-	1    0    0    -1
-$EndComp
-Text GLabel 5950 5000 0    60   Input ~ 0
+P 6750 6650
+F 0 "#PWR04" H 6750 6620 20  0001 C CNN
+F 1 "+9V" H 6750 6760 30  0000 C CNN
+F 2 "" H 6750 6650 60  0000 C CNN
+F 3 "" H 6750 6650 60  0000 C CNN
+	1    6750 6650
+	1    0    0    -1
+$EndComp
+Text GLabel 6900 5100 2    60   Input ~ 0
 PIN9V
 NoConn ~ 3750 5750
@@
 	1    0    0    -1
 $EndComp
-Text GLabel 5950 4700 0    60   Input ~ 0
+Text GLabel 6900 4700 2    60   Input ~ 0
 PIN5V
 Text GLabel 7500 5500 0    60   Input ~ 0
@@
 	9600 6500 9650 6500
 Wire Wire Line
-	5900 6300 5900 6800
+	5900 6200 5900 6800
 Wire Wire Line
 	1850 5500 1350 5500
@@
 	6300 1300 6000 1300
 Wire Wire Line
-	6150 5100 6100 5100
-Wire Wire Line
-	6000 5200 6900 5200
-Wire Wire Line
-	5900 6500 5550 6500
-Wire Wire Line
-	5550 6500 5550 6400
+	6000 5200 7300 5200
 Wire Wire Line
 	5900 5400 5950 5400
-Wire Wire Line
-	5950 5000 6150 5000
 Wire Wire Line
 	5700 3250 6250 3250
@@
 Connection ~ 9750 2850
 Wire Wire Line
-	8300 3000 7800 3000
+	7800 3000 8300 3000
 Connection ~ 8100 3000
 Wire Wire Line
@@
 	7300 6300 7300 6800
 Wire Wire Line
-	6650 6200 6650 6750
-Wire Wire Line
-	6650 6750 5900 6750
+	5900 6750 6900 6750
 Connection ~ 5900 6750
 Wire Wire Line
-	5800 6400 5800 6700
-Wire Wire Line
-	5800 6700 5900 6700
-Connection ~ 5900 6700
-Wire Wire Line
 	8450 6300 8950 6300
 Wire Wire Line
 	8950 6300 8950 6900
-Wire Wire Line
-	6900 5200 6900 4700
-Connection ~ 6100 5200
-Wire Wire Line
-	6100 4900 6150 4900
-Connection ~ 6100 5100
-Wire Wire Line
-	6100 4800 6150 4800
-Connection ~ 6100 4900
-Wire Wire Line
-	5950 4700 6150 4700
-Wire Wire Line
-	6100 4800 6100 5200
 Wire Wire Line
 	7650 4600 7500 4600
@@
 Connection ~ 9550 4900
 Connection ~ 9550 4800
-Wire Wire Line
-	6900 5100 6900 5000
-Connection ~ 6900 5000
-Connection ~ 6900 5100
-Wire Wire Line
-	6900 4900 6900 4800
-Connection ~ 6900 4800
 Connection ~ 6900 4900
-Wire Wire Line
-	6650 6600 6650 6500
 Connection ~ 6650 6500
-Connection ~ 6650 6600
-Wire Wire Line
-	6650 6400 6650 6300
 Connection ~ 6650 6300
 Connection ~ 6650 6400
@@
 Connection ~ 10400 6500
 Wire Wire Line
-	9650 6400 9650 6300
+	9650 6000 9650 6400
 Connection ~ 9650 6400
-Wire Wire Line
-	9650 6200 9650 6100
-Wire Wire Line
-	9650 6350 9650 6000
 Wire Wire Line
 	9650 6000 10400 6000
@@
 Connection ~ 9650 6300
 Connection ~ 5900 6600
+Connection ~ 5900 6500
+Wire Wire Line
+	6650 6500 6900 6500
+Wire Wire Line
+	6900 6500 6900 6750
+Wire Wire Line
+	7300 5200 7300 5000
+Wire Wire Line
+	7300 5000 6900 5000
+Connection ~ 6900 5000
+Wire Wire Line
+	6900 5000 6900 4800
+Wire Wire Line
+	6150 4700 6150 5200
+Connection ~ 6150 5200
+Connection ~ 6150 5100
+Connection ~ 6150 5000
+Connection ~ 6150 4900
+Connection ~ 6150 4800
+Wire Wire Line
+	6750 6650 6650 6650
+Wire Wire Line
+	6650 6650 6650 6600
+Wire Wire Line
+	6650 6500 6650 6300
+Connection ~ 5900 6300
 $EndSCHEMATC
