File: files/circuit/kicad/nixie.sch (KiCad schematic (older format))
At the start: 13 parts, among them IC2 74LC138, IC3 TLP627, IC4 TLP627, IC5 SN74141_K155NA, IC6 TLP627-4, IC7 TLP627-4

Commit message: 基板完成、発注版
Connections:
- net N0: now also IC5.15; no longer IC5.2
- net N1: now also IC5.14; no longer IC5.1
- net N2: now also IC5.8; no longer IC5.15
- net N3: now also IC5.9; no longer IC5.16
- net N4: now also IC5.10; no longer IC5.13
- net N5: now also IC5.11; no longer IC5.14
- net N6: now also IC5.13; no longer IC5.9
- net N7: now also IC5.16; no longer IC5.10
- net N8: now also IC5.1; no longer IC5.11
- net N9: now also IC5.2; no longer IC5.8
Changed lines of the file:
@@
 Sheet 2 8
 Title ""
-Date "7 sep 2014"
+Date "8 sep 2014"
 Rev ""
 Comp ""
@@
 Text Label 2550 6200 0    60   ~ 0
 PINPC2
-Text Label 4050 6000 0    60   ~ 0
+Text Label 5450 6000 0    60   ~ 0
 N0
-Text Label 4050 5900 0    60   ~ 0
+Text Label 5450 6100 0    60   ~ 0
 N1
-Text Label 5450 6000 0    60   ~ 0
+Text Label 4100 6600 0    60   ~ 0
 N2
+Text Label 5450 6600 0    60   ~ 0
+N3
+Text Label 5450 6500 0    60   ~ 0
+N4
+Text Label 5450 6400 0    60   ~ 0
+N5
+Text Label 5450 6200 0    60   ~ 0
+N6
 Text Label 5450 5900 0    60   ~ 0
-N3
-Text Label 5450 6200 0    60   ~ 0
-N4
-Text Label 5450 6100 0    60   ~ 0
-N5
-Text Label 5450 6600 0    60   ~ 0
-N6
-Text Label 5450 6500 0    60   ~ 0
 N7
-Text Label 5450 6400 0    60   ~ 0
+Text Label 4100 5900 0    60   ~ 0
 N8
-Text Label 4050 6600 0    60   ~ 0
+Text Label 4100 6000 0    60   ~ 0
 N9
 Text Label 2850 4200 0    60   ~ 0
